File: power_board_24V/power_board_24V.kicad_sch (KiCad schematic)
At the start: 40 parts, among them J1 Conn_01x02_Pin, J10 Conn_01x02_Pin, J11 Conn_01x02_Pin, J12 Conn_01x02_Pin, J13 Conn_01x02_Pin, J14 Conn_01x02_Pin, J2 Conn_01x02_Pin, J3 Conn_01x02_Pin, J4 Conn_01x02_Pin, J5 Conn_01x02_Pin, J6 Conn_01x02_Pin, J7 Conn_01x02_Pin, J8 Conn_01x02_Pin, J9 Conn_01x02_Pin, K1 A31CCQ24VDC1D, Q1 2N7000, U1 INA226

Commit message: 24V基板　シミュレーションの回路を実際の回路に適応した．また，放電抵抗を取り外した． スロースタート用コンデンサの常時放電抵抗があることにより，可変抵抗の抵抗値を上げた際にスロースタートが解除されないことが分かった．放電用ダイオードもあるため，放電抵抗は消した．
Parts:
- added D6: SM340A, Diode_SMD:D_SMA_Handsoldering, symbol Device:D_Schottky
- added Q2: 2SA1015, Package_TO_SOT_THT:TO-92_Inline, symbol Transistor_BJT:2SA1015
- added R11, R12: 47k, symbol Device:R
- added R13: 220k, symbol Device:R
Connections:
- net at C4.1, D4.2 (A), DZ1.1 (K)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: now also R13.2
- net at K1.85, Q1.3 (D): now also R12.2
- net at D4.1 (K), J13.2 (Pin_2), K1.86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: now also D6.2 (A), Q2.1 (E), R11.1; no longer R10.1
- new net: Q2.2 (C), R13.1
- new net: Q2.3 (B), R11.2, R12.1
- new net: D6.1 (K), R10.1
Other:
- note added: "フットプリント要チェック"
- moved on the sheet: C4, D1, D3, D4, DZ1, J10, J11, J12, J14, J2, J3, J4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

Commit message: 24V基板　フットプリント割当まで完了
Parts:
- removed C4: 10u, Capacitor_THT:C_Disc_D6.0mm_W4.4mm_P5.00mm, symbol Device:C
- removed J10, J11, J14, J2, J3, J4, J5, J6, J7, J9: Conn_01x02_Pin, OU_Conn:AMASS_XT30U-F, symbol Connector:Conn_01x02_Pin
- removed Q1: 2N7000, Package_TO_SOT_THT:TO-92_Inline, symbol Transistor_FET:2N7000
- added C4: 10u, Capacitor_THT:CP_Radial_D5.0mm_P2.00mm, symbol Device:C_Polarized
- added D6, D7: SMBJ30CA, PCM_Diode_SMD_AKL:D_SMB_TVS, symbol PCM_Diode_TVS_AKL:SMBJ30CA
- added J11, J14, J2, J3, J4, J5, J6, J7, J8, J9: Conn_01x02_Socket, OU_connector:AMASS_XT30U-F_1x02_P5.0mm_Vertical, symbol Connector:Conn_01x02_Socket
- added J15: Conn_01x04_Pin, OU_connector:DF1EC-4P-2.5DSA, symbol Connector:Conn_01x04_Pin
- added Q2: BS170, Package_TO_SOT_THT:TO-92_Inline, symbol Transistor_FET:BS170
- added R13, R15: 4.7k, Resistor_SMD:R_0603_1608Metric, symbol Device:R
- D1, D2, D3: Buy_URL (none) -> https://akizukidenshi.com/catalog/g/https://akizukidenshi.c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
- D4: footprint Diode_THT:D_DO-35_SOD27_P2.54mm_Vertical_CathodeUp -> Diode_THT:D_DO-34_SOD68_P2.54mm_Vertical_CathodeUp; Buy_URL (none) -> https://akizukidenshi.com/catalog/g/g116603/; MPN_URL https://akizukidenshi.com/catalog/g/g100941/ -> (none)
- D5: renamed from D6; Buy_URL (none) -> https://akizukidenshi.com/catalog/g/g109915/
- DZ1: Buy_URL (none) -> https://akizukidenshi.com/catalog/g/g115721/
- F1: footprint (none) -> OU_Fuse:FUC-03A_20mm; Buy_URL (none) -> https://akizukidenshi.com/catalog/g/g107131/; Set_Parts (none) -> https://akizukidenshi.com/catalog/g/g110521/
- F2: footprint (none) -> OU_Fuse:3557-15_KEY; Buy_URL (none) -> https://akizukidenshi.com/catalog/g/g118221/; Set_Parts (none) -> https://akizukidenshi.com/catalog/g/g118223/
- J1: footprint (none) -> OU_connector:AMASS_XT60PW-M_1x02_P7.20mm_Horizontal; Buy_URL (none) -> https://akizukidenshi.com/catalog/g/g118156/
- J10: renamed from J8; footprint (none) -> OU_connector:DF1EC-2P-2.5DSA
- J12, J13: footprint (none) -> OU_connector:DF1E-2P-2.5DS
- K1: Buy_URL (none) -> https://www.digikey.com/en/products/detail/cit-relay-and-sw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; MPN A31CCQ24VDC1D, DZ85AB-5-PCB -> (none); MPN_URL https://eleshop.jp/shop/g/g2292976/?srsltid=AfmBOor25f7k4UF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 -> (none); Set_Parts (none) -> https://eleshop.jp/shop/g/g2292976/?srsltid=AU7gw4WNeVHQNYN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
- NT1: footprint (none) -> NetTie:NetTie-2_SMD_Pad2.0mm
- Q1: renamed from Q2; Buy_URL (none) -> https://akizukidenshi.com/catalog/g/g117091/
- R1, R2, R7: footprint (none) -> Resistor_THT:R_Axial_DIN0207_L6.3mm_D2.5mm_P2.54mm_Vertical; Buy_URL (none) -> https://akizukidenshi.com/catalog/g/g125752/
- R10: renamed from R13; footprint (none) -> Resistor_SMD:R_0603_1608Metric
- R11, R12, R8, R9: footprint (none) -> Resistor_SMD:R_0603_1608Metric
- R14: renamed from R10; Buy_URL (none) -> https://akizukidenshi.com/catalog/g/g103991/; MPN_URL https://akizukidenshi.com/catalog/g/g103991/ -> (none)
- RV1: footprint (none) -> OU_Reg:GF063P; Buy_URL (none) -> https://akizukidenshi.com/catalog/g/g114913/
Connections:
- net +24V_CTRL: now also J11.2 (Pin_2), J14.2 (Pin_2), J7.2 (Pin_2), J8.2 (Pin_2), J9.2 (Pin_2)
- net +24V_DRV: now also D6.2 (A), J2.2 (Pin_2), J3.2 (Pin_2), J4.2 (Pin_2), J5.2 (Pin_2), J6.2 (Pin_2)
- net +3.3V: now also J15.3 (Pin_3), R13.1, R15.1
- net GND: now also J11.1 (Pin_1), J14.1 (Pin_1), J15.1 (Pin_1), J7.1 (Pin_1), J8.1 (Pin_1), J9.1 (Pin_1)
- net GNDPWR: now also C4.2, D6.1 (K), D7.1 (K), J2.1 (Pin_1), J3.1 (Pin_1), J4.1 (Pin_1), J5.1 (Pin_1), J6.1 (Pin_1), Q2.3 (S)
- net I2C_SCL: now also J15.2 (Pin_2), R15.2
- net I2C_SDA: now also J15.4 (Pin_4), R13.2
- net at D4.2 (A), DZ1.1 (K), J12.1 (Pin_1)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: now also C4.1, Q2.2 (G)
- net at K1.85, R12.2: now also Q2.1 (D)
- net at F1.2, F2.1, R4.1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: no longer J10.2 (Pin_2)
- net at J1.2 (Pin_2), R2.1, R4.4: now also D7.2 (A)
- net at F2.2, J13.1 (Pin_1), K1.87: now also J10.2 (Pin_2)
Other:
- note added: "通信"
- moved on the sheet: C1, C2, C3, D3, D4, D5, DZ1, F1, F2, J10, J12, J13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

Commit message: 24V基板　基板完成 ver 1.0
Parts:
- renumbered C3 to C1, C1 to C3, D7 to D1, D5 to D3, D6 to D5, D1 to D6, D3 to D7, J10 to J1, J7 to J10, J8 to J11, J9 to J12, J11 to J13, J1 to J2, J13 to J3, J12 to J4, J2 to J5, J3 to J6, J4 to J7, J5 to J8, J6 to J9, R4 to R1, R8 to R11, R1 to R12, R7 to R13, R13 to R14, R6 to R3, R3 to R4, R14 to R6, R11 to R7, R12 to R8
Connections:
- net GND: now also D7.1 (K)
- net GNDPWR: no longer D7.1 (K)
Other:
- note added: "24Vフロントエンド"
- moved on the sheet: NT1
