File: servo_control_board/servo_control_board.kicad_pcb (KiCad board)
At the start: 2 copper layers, 85 x 35 mm, 40 parts, among them J1 Conn_01x03_Pin, J2 Conn_01x03_Pin, J3 Conn_01x03_Pin, J4 Conn_01x03_Pin, J5 Conn_01x03_Pin, J6 Conn_01x03_Pin, J7 Conn_01x02_Pin, U1 H11L1M, U2 H11L1M, U3 H11L1M, U4 H11L1M

Commit message: サーボ制御基板　コネクタをJST PAに変更
Parts:
- J1, J2: footprint OU_connector:DF1E-3P-2.5DS -> OU_connector:S03B-PASK-2
- moved J2 3.57 mm to (82.5, 28.7)
- moved J1 3.56 mm to (52.1, 28.7)
Connections:
- R1 pad 1: Net-(J1-Pin_3) -> Net-(J1-Pin_1)
- R2 pad 1: Net-(J2-Pin_3) -> Net-(J2-Pin_1)
- R3 pad 1: Net-(J1-Pin_1) -> Net-(J1-Pin_3)
- R4 pad 1: Net-(J2-Pin_1) -> Net-(J2-Pin_3)
- TP1 pad 1: Net-(J1-Pin_3) -> Net-(J1-Pin_1)
- TP2 pad 1: Net-(J2-Pin_3) -> Net-(J2-Pin_1)
- TP4 pad 1: Net-(J1-Pin_1) -> Net-(J1-Pin_3)
- TP5 pad 1: Net-(J2-Pin_1) -> Net-(J2-Pin_3)
Routing:
- net Net-(J1-Pin_3): track 15.0 -> 18.0 mm
- net Net-(J2-Pin_3): track 15.0 -> 17.8 mm
- net Net-(J2-Pin_1): track 15.0 -> 17.7 mm
- net Net-(J1-Pin_1): track 15.3 -> 17.8 mm
Other:
- board text added: "2026/10/01 Designed by E.Yoshioka"
- board text added: "ver 0.2"
- board text removed: "2026/09/24 Designed by E.Yoshioka"
- board text removed: "ver 0.1"

Commit message: サーボ制御基板　シルクを一部修正，ver 1.0
Other:
- board text added: "2026/10/10 Designed by E.Yoshioka"
- board text added: "ver 1.0"
- board text removed: "2026/10/01 Designed by E.Yoshioka"
- board text removed: "ver 0.2"
Changed lines of the file:
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@@
+	)
+	(gr_rect
+		(start 23.154 32.552)
+		(end 28.154 37.552)
+		(stroke
+			(width 0)
+			(type solid)
+		)
+		(fill yes)
+		(layer "B.SilkS")
 	)
 	(gr_rect
@@
 		)
 	)
-	(gr_text "ver 0.2"
+	(gr_text "ver 1.0"
 		(at 28 28.392 0)
 		(layer "F.SilkS")
@@
 		)
 	)
-	(gr_text "2026/10/01\nDesigned by\nE.Yoshioka"
+	(gr_text "2026/10/10\nDesigned by\nE.Yoshioka"
 		(at 48 23.5 0)
 		(layer "B.SilkS")
