File: servo_power_board/servo_power_board.kicad_pcb (KiCad board)
At the start: 2 copper layers, 85 x 55 mm, 25 parts, among them J1 Conn_01x02_Pin, J2 Conn_01x02_Socket, J3 Conn_01x02_Pin, J4 Conn_01x02_Socket, J5 Conn_01x02_Socket, J6 Conn_01x02_Socket, U1 YDS512F

Commit message: サーボ電源基板　基板にテストポイントを追加，ver 0.2
Parts:
- added TP1: TestPoint, TestPoint:TestPoint_THTPad_D2.0mm_Drill1.0mm, F.Cu at (89.9, 21.8)
- added TP2: TestPoint_Probe, TestPoint:TestPoint_THTPad_D2.0mm_Drill1.0mm, F.Cu at (96.0, 73.2)
Routing:
- net Net-(J3-Pin_2): track 104.1 -> 114.6 mm
- net GND: vias 111 -> 113
Other:
- board text added: "+SERVO"
- board text added: "BoardID: TS26-PWR -SRV ver 0.2"
- board text added: "GND"
- board text removed: "BoardID: TS26-PWR -SRV ver 0.1"

Commit message: サーボ電源基板　シルクの向きが間違っていたのを修正，ver0.3
Other:
- board text added: "BoardID: TS26-PWR -SRV ver 0.3"
- board text removed: "BoardID: TS26-PWR -SRV ver 0.2"
Changed lines of the file:
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@@
 		(layer "Edge.Cuts")
 	)
-	(gr_text "BoardID:\n TS26-PWR\n -SRV\n\nver 0.2"
+	(gr_text "BoardID:\n TS26-PWR\n -SRV\n\nver 0.3"
 		(at 34.5 60.5 0)
 		(layer "F.SilkS")
@@
 	)
 	(gr_text "2026/09/20\nDesigned by E.Yoshioka"
-		(at 83 45.9 270)
+		(at 83 45.9 0)
 		(layer "B.SilkS")
 		(effects
