File: servo_power_board/servo_power_board.kicad_pcb (KiCad board)
At the start: 2 copper layers, 85 x 55 mm, 27 parts, among them J1 Conn_01x02_Pin, J2 Conn_01x02_Socket, J3 Conn_01x02_Pin, J4 Conn_01x02_Socket, J5 Conn_01x02_Socket, J6 Conn_01x02_Socket, U1 YDS512F

Commit message: サーボ電源基板　シルクを一部修正，ネジ下のベタを削除，ver 1.0
Routing:
- net GND: vias 113 -> 109
Other:
- board text added: "2026/10/10 Designed by E.Yoshioka"
- board text added: "BoardID: TS26-PWR -SRV ver 1.0"
- board text removed: "2026/09/20 Designed by E.Yoshioka"
- board text removed: "BoardID: TS26-PWR -SRV ver 0.3"
Changed lines of the file:
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@@
+	)
+	(gr_rect
+		(start 88.646 37.72)
+		(end 96.646 45.72)
+		(stroke
+			(width 0)
+			(type solid)
+		)
+		(fill yes)
+		(layer "B.SilkS")
 	)
 	(gr_rect
@@
 		(layer "Edge.Cuts")
 	)
-	(gr_text "BoardID:\n TS26-PWR\n -SRV\n\nver 0.3"
+	(gr_text "BoardID:\n TS26-PWR\n -SRV\n\nver 1.0"
 		(at 34.5 60.5 0)
 		(layer "F.SilkS")
@@
 		)
 	)
-	(gr_text "2026/09/20\nDesigned by E.Yoshioka"
+	(gr_text "2026/10/10\nDesigned by E.Yoshioka"
 		(at 83 45.9 0)
 		(layer "B.SilkS")
@@
 	)
 	(via
-		(at 90 45)
-		(size 0.8)
-		(drill 0.4)
-		(layers "F.Cu" "B.Cu")
-		(free yes)
-		(net "GND")
-	)
-	(via
 		(at 50 50)
 		(size 0.8)
@@
 	)
 	(via
-		(at 90 40)
-		(size 0.8)
-		(drill 0.4)
-		(layers "F.Cu" "B.Cu")
-		(free yes)
-		(net "GND")
-	)
-	(via
 		(at 80 52.25)
 		(size 0.8)
@@
 	)
 	(via
-		(at 95 40)
-		(size 0.8)
-		(drill 0.4)
-		(layers "F.Cu" "B.Cu")
-		(free yes)
-		(net "GND")
-	)
-	(via
 		(at 70 35)
-		(size 0.8)
-		(drill 0.4)
-		(layers "F.Cu" "B.Cu")
-		(free yes)
-		(net "GND")
-	)
-	(via
-		(at 95 45)
 		(size 0.8)
 		(drill 0.4)
@@
 		(polygon
 			(pts
+				(xy 96 30.5) (xy 104 30.5) (xy 104 38.5) (xy 96 38.5)
+			)
+		)
+	)
+	(zone
+		(layers "F.Cu" "B.Cu")
+		(hatch edge 0.5)
+		(connect_pads yes
+			(clearance 0)
+		)
+		(min_thickness 0.25)
+		(keepout
+			(tracks allowed)
+			(vias allowed)
+			(pads allowed)
+			(copperpour not_allowed)
+			(footprints allowed)
+		)
+		(placement
+			(enabled no)
+			(sheetname "")
+		)
+		(fill
+			(thermal_gap 0.5)
+			(thermal_bridge_width 0.5)
+			(island_removal_mode 0)
+		)
+		(polygon
+			(pts
 				(xy 97 20) (xy 105 20) (xy 105 28) (xy 97 28)
 			)
 		)
+	)
+	(zone
+		(layers "F.Cu" "B.Cu")
+		(hatch edge 0.5)
+		(connect_pads yes
+			(clearance 0)
+		)
+		(min_thickness 0.25)
+		(keepout
+			(tracks allowed)
+			(vias allowed)
+			(pads allowed)
+			(copperpour not_allowed)
+			(footprints allowed)
+		)
+		(placement
+			(enabled no)
+			(sheetname "")
+		)
+		(fill
+			(thermal_gap 0.5)
+			(thermal_bridge_width 0.5)
+			(island_removal_mode 0)
+		)
+		(polygon
+			(pts
+				(xy 96 56.5) (xy 104 56.5) (xy 104 64.5) (xy 96 64.5)
+			)
+		)
