File: 24v_power_board/24v_power_board.kicad_sch (KiCad schematic)
At the start: 54 parts, among them J1 Conn_01x02_Pin, J10 Conn_01x02_Socket, J11 Conn_01x02_Socket, J12 Conn_01x02_Socket, J13 Conn_01x02_Socket, J14 Conn_01x02_Socket, J15 Conn_01x04_Pin, J2 Conn_01x02_Pin, J3 Conn_01x02_Pin, J4 Conn_01x02_Pin, J5 Conn_01x02_Socket, J6 Conn_01x02_Socket, J7 Conn_01x02_Socket, J8 Conn_01x02_Socket, J9 Conn_01x02_Socket, K1 A31CCQ24VDC1D, Q1 2SA1015, Q2 BS170, U1 INA226

Commit message: 24V基板　PAコネクタに変更，ver 0.7
Parts:
- J1: footprint OU_connector:DF1EC-2P-2.5DSA -> OU_connector:B02B-PASK-1
- J15: footprint OU_connector:DF1EC-4P-2.5DSA -> OU_connector:B04B-PASK-1
- J3, J4: footprint OU_connector:DF1E-2P-2.5DS -> OU_connector:S02B-PASK-2
Changed lines of the file:
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@@
 			)
 		)
-		(property "Footprint" "OU_connector:DF1EC-2P-2.5DSA"
+		(property "Footprint" "OU_connector:B02B-PASK-1"
 			(at 148.59 25.4 0)
 			(hide yes)
@@
 			)
 		)
-		(property "Description" "DF1EC-2P-2.5DSA"
+		(property "Description" "B02B-PASK-1"
 			(at 148.59 25.4 0)
 			(hide yes)
@@
 			)
 		)
-		(property "Footprint" "OU_connector:DF1EC-4P-2.5DSA"
+		(property "Footprint" "OU_connector:B04B-PASK-1"
 			(at 189.23 139.7 0)
 			(hide yes)
@@
 			)
 		)
-		(property "Description" "DF1EC-4P-2.5DSA"
+		(property "Description" "B04B-PASK-1"
 			(at 189.23 139.7 0)
 			(hide yes)
@@
 			)
 		)
-		(property "Footprint" "OU_connector:DF1E-2P-2.5DS"
+		(property "Footprint" "OU_connector:S02B-PASK-2"
 			(at 161.29 44.45 0)
 			(hide yes)
@@
 			)
 		)
-		(property "Description" "DF1E-2P-2.5DS"
+		(property "Description" "S02B-PASK-2"
 			(at 161.29 44.45 0)
 			(hide yes)
@@
 			)
 		)
-		(property "Footprint" "OU_connector:DF1E-2P-2.5DS"
+		(property "Footprint" "OU_connector:S02B-PASK-2"
 			(at 157.48 96.52 0)
 			(hide yes)
@@
 			)
 		)
-		(property "Description" "DF1E-2P-2.5DS"
+		(property "Description" "S02B-PASK-2"
 			(at 157.48 96.52 0)
 			(hide yes)

Commit message: 24V基板　再度DF1Eに変更，ver 0.8 一度PAコネクタに変更したが，在庫数の関係で3ピンのみPAにすることにしたため，他はDF1Eに戻した．
Parts:
- J1: footprint OU_connector:B02B-PASK-1 -> OU_connector:DF1EC-2P-2.5DSA
- J15: footprint OU_connector:B04B-PASK-1 -> OU_connector:DF1EC-4P-2.5DSA
- J3, J4: footprint OU_connector:S02B-PASK-2 -> OU_connector:DF1E-2P-2.5DS
Changed lines of the file:
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@@
 			)
 		)
-		(property "Footprint" "OU_connector:B02B-PASK-1"
+		(property "Footprint" "OU_connector:DF1EC-2P-2.5DSA"
 			(at 148.59 25.4 0)
 			(hide yes)
@@
 			)
 		)
-		(property "Footprint" "OU_connector:B04B-PASK-1"
+		(property "Footprint" "OU_connector:DF1EC-4P-2.5DSA"
 			(at 189.23 139.7 0)
 			(hide yes)
@@
 			)
 		)
-		(property "Footprint" "OU_connector:S02B-PASK-2"
+		(property "Footprint" "OU_connector:DF1E-2P-2.5DS"
 			(at 161.29 44.45 0)
 			(hide yes)
@@
 			)
 		)
-		(property "Footprint" "OU_connector:S02B-PASK-2"
+		(property "Footprint" "OU_connector:DF1E-2P-2.5DS"
 			(at 157.48 96.52 0)
 			(hide yes)
