File: 24v_power_board/24v_power_board.kicad_pcb (KiCad board)
At the start: 2 copper layers, 100 x 60 mm, 60 parts, among them J1 Conn_01x02_Pin, J10 Conn_01x02_Socket, J11 Conn_01x02_Socket, J12 Conn_01x02_Socket, J13 Conn_01x02_Socket, J14 Conn_01x02_Socket, J15 Conn_01x04_Pin, J2 Conn_01x02_Pin, J3 Conn_01x02_Pin, J4 Conn_01x02_Pin, J5 Conn_01x02_Socket, J6 Conn_01x02_Socket, J7 Conn_01x02_Socket, J8 Conn_01x02_Socket, J9 Conn_01x02_Socket, K1 A31CCQ24VDC1D, Q1 2SA1015, Q2 BS170, U1 INA226

Commit message: 24V基板　再度DF1Eに変更，ver 0.8 一度PAコネクタに変更したが，在庫数の関係で3ピンのみPAにすることにしたため，他はDF1Eに戻した．
Parts:
- J1: footprint OU_connector:B02B-PASK-1 -> OU_connector:DF1EC-2P-2.5DSA
- J15: footprint OU_connector:B04B-PASK-1 -> OU_connector:DF1EC-4P-2.5DSA
- J3, J4: footprint OU_connector:S02B-PASK-2 -> OU_connector:DF1E-2P-2.5DS
- moved J15 4.02 mm to (59.1, 21.6)
- moved J3 3.78 mm to (75.9, 65.0)
- moved J4 3.06 mm to (94.0, 26.9)
- moved R11 2.43 mm to (96.5, 23.6)
- moved J1 2.12 mm to (58.7, 58.2)
Routing:
- net Net-(J1-Pin_2): track 56.1 -> 61.2 mm
- net /I2C_SCL: track 11.1 -> 13.5 mm
- net Net-(D4-A): track 49.7 -> 47.5 mm
- net Net-(D3-A): track 62.6 -> 64.4 mm
- net +3.3V: track 12.1 -> 13.1 mm
- net Net-(J4-Pin_2): track 1.87 -> 2.49 mm
Other:
- board text added: "BoardID: TS26-PWR-MAIN ver 0.8"
- board text removed: "BoardID: TS26-PWR-MAIN ver 0.7"

Commit message: 24V基板　リレーのフットプリントにミスがあったため，それを修正，ver 0.9
Parts:
- turned K1 to 90 degrees
Routing:
- net Net-(Q2-D): track 30.4 -> 45.8 mm
- net Net-(D3-A): track 64.4 -> 69.1 mm
- net Net-(J1-Pin_2): track 61.2 -> 61.7 mm
- net GNDPWR: vias 46 -> 52
Other:
- board text added: "BoardID: TS26-PWR-MAIN ver 0.9"
- board text removed: "BoardID: TS26-PWR-MAIN ver 0.8"

Commit message: 24V基板　シルクの一部修正，ver 1.0
Other:
- board text added: "2026/10/10 Designed by E.Yoshioka"
- board text added: "BoardID: TS26-PWR-MAIN ver 1.0"
- board text removed: "2026/09/23 Designed by E.Yoshioka"
- board text removed: "BoardID: TS26-PWR-MAIN ver 0.9"
Changed lines of the file:
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@@
 		(tags "connector Hirose DF1E right-angle 2pin 2.5mm")
 		(property "Reference" "J3"
-			(at 1.25 -12.6 180)
+			(at 6.604 2.54 180)
 			(layer "F.SilkS")
 			(effects
@@
 		(tags "capacitor")
 		(property "Reference" "C1"
-			(at 0 1.43 90)
+			(at 2.527 0 90)
 			(layer "B.SilkS")
 			(effects
@@
 		(layer "Edge.Cuts")
 	)
-	(gr_text "BoardID:\n TS26-PWR-MAIN\n\nver 0.9"
+	(gr_text "BoardID:\n TS26-PWR-MAIN\n\nver 1.0"
 		(at 35.56 28.956 0)
 		(layer "F.SilkS")
@@
 		)
 	)
-	(gr_text "2026/09/23\nDesigned by E.Yoshioka"
+	(gr_text "2026/10/10\nDesigned by E.Yoshioka"
 		(at 61 40 0)
 		(layer "B.SilkS")

Commit message: 24V基板　シリアルコード用QRを追加，ver 1.1
Other:
- board text added: "BoardID: TS26-PWR-MAIN ver 1.1"
- board text removed: "BoardID: TS26-PWR-MAIN ver 1.0"
Changed lines of the file:
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@@
+	)
+	(gr_rect
+		(start 55.372 45.276)
+		(end 63.372 53.276)
+		(stroke
+			(width 0)
+			(type solid)
+		)
+		(fill yes)
+		(layer "B.SilkS")
 	)
 	(gr_rect
@@
 		(layer "Edge.Cuts")
 	)
-	(gr_text "BoardID:\n TS26-PWR-MAIN\n\nver 1.0"
+	(gr_text "BoardID:\n TS26-PWR-MAIN\n\nver 1.1"
 		(at 35.56 28.956 0)
 		(layer "F.SilkS")
@@
 	)
 	(gr_text "2026/10/10\nDesigned by E.Yoshioka"
-		(at 61 40 0)
+		(at 63.5 39.116 0)
 		(layer "B.SilkS")
 		(effects

Commit message: 24V電源基板　プリチャージ抵抗と直列にポリスイッチを追加，ver 1.2 非常停止スイッチ接続端子がどちらもONになった場合，リレーがオンにならず，プリチャージ抵抗に電流が流れ続ける可能性があった．そこでポリスイッチを直列に接続することで，プリチャージ抵抗に電流が流れ続けた場合に電流が遮断されるようにした．
Parts:
- added F3: MF-RX065, Fuse:Fuse_BelFuse_0ZRE0016FF_L9.9mm_W3.8mm, F.Cu at (82.3, 55.3)
- moved D3 4.06 mm to (83.8, 59.9)
Connections:
- D4 pad 1: Net-(D3-A) -> Net-(D4-K)
- J3 pad 2: Net-(D3-A) -> Net-(D4-K)
- K1 pad 86: Net-(D3-A) -> Net-(D4-K)
- Q1 pad 1: Net-(D3-A) -> Net-(D4-K)
- R7 pad 1: Net-(D3-A) -> Net-(D4-K)
- R9 pad 1: Net-(D3-A) -> Net-(D4-K)
Routing:
- net Net-(D4-K): track 0.00 -> 69.7 mm
- net Net-(D3-A): track 69.1 -> 7.29 mm
- net Net-(D3-K): track 7.62 -> 3.57 mm
- net GNDPWR: vias 52 -> 51
Other:
- board text added: "2026/10/11 Designed by E.Yoshioka"
- board text added: "BoardID: TS26-PWR-MAIN ver 1.2"
- board text removed: "2026/10/10 Designed by E.Yoshioka"
- board text removed: "BoardID: TS26-PWR-MAIN ver 1.1"

Commit message: 24V電源基板　ポリスイッチを変更，ver 1.3 変更前のポリスイッチはトリップ電流や時間が大きく，電流が遮断される前にプリチャージ抵抗や基板にダメージが入る可能性があった．そのため，トリップ電流や時間が小さいものに変更した．
Parts:
- F3: value MF-RX065 -> MF-RX030; footprint Fuse:Fuse_BelFuse_0ZRE0016FF_L9.9mm_W3.8mm -> Fuse:Fuse_Bourns_MF-RHT050
Routing:
- net Net-(D4-K): track 69.7 -> 65.5 mm
Other:
- board text added: "2026/10/12 Designed by E.Yoshioka"
- board text added: "BoardID: TS26-PWR-MAIN ver 1.3"
- board text removed: "2026/10/11 Designed by E.Yoshioka"
- board text removed: "BoardID: TS26-PWR-MAIN ver 1.2"
