File: Nucleo-F303K8_control_board/Nucleo-F303K8_control_board.kicad_pcb (KiCad board)
At the start: 2 copper layers, 55 x 70 mm, 33 parts, among them J1 Conn_01x02_Pin, J10 Conn_01x04_Pin, J11 Conn_01x04_Pin, J2 Conn_01x03_Pin, J3 Conn_01x03_Pin, J4 Conn_01x02_Pin, J5 Conn_01x02_Pin, J6 Conn_01x04_Pin, J7 Conn_01x03_Pin, J8 Conn_01x03_Pin, J9 Conn_01x03_Pin, U1 NUCLEO-F303K8, U2 MCP2562-E-P

Commit message: F303K8基板　シルクを一部修正，ver 1.0
Other:
- board text added: "2026/10/10 Designed by E.Yoshioka"
- board text added: "ver 1.0"
- board text removed: "2026/10/05 Designed by E.Yoshioka"
- board text removed: "ver 0.2"
Changed lines of the file:
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@@
 		(tags "LED")
 		(property "Reference" "D1"
-			(at 0 -4.064 90)
+			(at 5.08 -1.27 180)
 			(layer "F.SilkS")
 			(effects
@@
 		)
 	)
-	(gr_text "ver 0.2"
+	(gr_text "ver 1.0"
 		(at 27.432 26.924 0)
 		(layer "F.SilkS")
@@
 		)
 	)
-	(gr_text "2026/10/05\nDesigned by E.Yoshioka"
+	(gr_text "5V"
+		(at 66.04 24.638 90)
+		(layer "F.SilkS" knockout)
+		(effects
+			(font
+				(size 1.5 1.5)
+				(thickness 0.3)
+				(bold yes)
+			)
+			(justify left)
+		)
+	)
+	(gr_text "2026/10/10\nDesigned by E.Yoshioka"
 		(at 73 57 270)
 		(layer "B.SilkS")

Commit message: F303K8基板　QRを追加，ver 1.1
Other:
- board text added: "ver 1.1"
- board text removed: "ver 1.0"
Changed lines of the file:
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@@
+	)
+	(gr_rect
+		(start 32.552 65.318)
+		(end 37.552 70.318)
+		(stroke
+			(width 0)
+			(type solid)
+		)
+		(fill yes)
+		(layer "B.SilkS")
 	)
 	(gr_rect
@@
 		)
 	)
-	(gr_text "ver 1.0"
+	(gr_text "ver 1.1"
 		(at 27.432 26.924 0)
 		(layer "F.SilkS")
