File: ESP32-DevKitC_control_board/ESP32-DevKitC_control_board.kicad_sch (KiCad schematic)
At the start: 33 parts, among them J1 Conn_01x02_Pin, J10 Conn_01x03_Pin, J11 Conn_01x03_Pin, J2 Conn_01x03_Pin, J3 Conn_01x03_Pin, J4 Conn_01x02_Pin, J5 Conn_01x02_Pin, J6 Conn_01x02_Pin, J7 Conn_01x04_Pin, J8 Conn_01x03_Pin, J9 Conn_01x03_Pin, U1 MCP2562-E-P, U2 ESP32-DevKitC

Commit message: ESP32基板　シルクを一部修正，3Dモデルを追加，ver 1.0
Parts:
- renumbered C2 to C1, C1 to C2, D4 to D1, J2 to J1, J3 to J2, J1 to J3, J5 to J4, J4 to J5, J7 to J6, J6 to J7, R12 to R1, R9 to R10, R10 to R11, R11 to R12, R1 to R2, R2 to R3, R3 to R4, R4 to R5, R5 to R6, R6 to R7, R7 to R8, R8 to R9
