File: ESP32-DevKitC_control_board/ESP32-DevKitC_control_board.kicad_pcb (KiCad board)
At the start: 2 copper layers, 85 x 60 mm, 39 parts, among them J1 Conn_01x02_Pin, J10 Conn_01x03_Pin, J11 Conn_01x03_Pin, J2 Conn_01x03_Pin, J3 Conn_01x03_Pin, J4 Conn_01x02_Pin, J5 Conn_01x02_Pin, J6 Conn_01x02_Pin, J7 Conn_01x04_Pin, J8 Conn_01x03_Pin, J9 Conn_01x03_Pin, U1 MCP2562-E-P, U2 ESP32-DevKitC

Commit message: ESP32基板　PWMの通し番号も1スタートに変更，ver 0.4
Connections:
- J2 pad 1: /PWM1 -> /PWM2
- J2 pad 3: /PWM0 -> /PWM1
- J3 pad 1: /PWM3 -> /PWM4
- J3 pad 3: /PWM2 -> /PWM3
- U2 pad 10: /PWM3 -> /PWM4
- U2 pad 11: /PWM1 -> /PWM2
- U2 pad 12: /PWM0 -> /PWM1
- U2 pad 9: /PWM2 -> /PWM3
Routing:
- net /PWM4: track 0.00 -> 32.3 mm
- net /PWM0: track 27.1 -> 0.00 mm
- net /PWM3: track 32.3 -> 25.9 mm
- net /PWM1: track 26.5 -> 27.1 mm
- net /PWM2: track 25.9 -> 26.5 mm
Other:
- board text added: "BoardID: TS26-CTRL-ESP32 ver 0.4"
- board text added: "PW2,4"
- board text added: "PWM1,2"
- board text added: "PWM3.4"
- board text removed: "BoardID: TS26-CTRL-ESP32 ver 0.3"
- board text removed: "PW0,2"
- board text removed: "PWM0,1"
- board text removed: "PWM2,3"
Changed lines of the file:
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@@
 			(layers "*.Cu" "*.Mask")
 			(remove_unused_layers no)
-			(net "/PWM1")
+			(net "/PWM2")
 			(pinfunction "Pin_1_1")
 			(pintype "passive")
@@
 			(layers "*.Cu" "*.Mask")
 			(remove_unused_layers no)
-			(net "/PWM0")
+			(net "/PWM1")
 			(pinfunction "Pin_3_3")
 			(pintype "passive")
@@
 			(layers "*.Cu" "*.Mask")
 			(remove_unused_layers no)
-			(net "/PWM2")
+			(net "/PWM3")
 			(pinfunction "DAC_1/ADC2_CH8/GPIO25_9")
 			(pintype "bidirectional")
@@
 			(layers "*.Cu" "*.Mask")
 			(remove_unused_layers no)
-			(net "/PWM3")
+			(net "/PWM4")
 			(pinfunction "DAC_2/ADC2_CH9/GPIO26_10")
 			(pintype "bidirectional")
@@
 			(layers "*.Cu" "*.Mask")
 			(remove_unused_layers no)
-			(net "/PWM1")
+			(net "/PWM2")
 			(pinfunction "ADC2_CH7/GPIO27_11")
 			(pintype "bidirectional")
@@
 			(layers "*.Cu" "*.Mask")
 			(remove_unused_layers no)
-			(net "/PWM0")
+			(net "/PWM1")
 			(pinfunction "MTMS/GPIO14/ADC2_CH6_12")
 			(pintype "bidirectional")
@@
 			(layers "*.Cu" "*.Mask")
 			(remove_unused_layers no)
-			(net "/PWM3")
+			(net "/PWM4")
 			(pinfunction "Pin_1_1")
 			(pintype "passive")
@@
 			(layers "*.Cu" "*.Mask")
 			(remove_unused_layers no)
-			(net "/PWM2")
+			(net "/PWM3")
 			(pinfunction "Pin_3_3")
 			(pintype "passive")
@@
 		)
 	)
-	(gr_text "BoardID:\n TS26-CTRL-ESP32\n\nver 0.3"
+	(gr_text "BoardID:\n TS26-CTRL-ESP32\n\nver 0.4"
 		(at 39 24.5 0)
 		(layer "F.SilkS")
@@
 		)
 	)
-	(gr_text "PW0,2"
+	(gr_text "PW1,3"
 		(at 98 48 0)
 		(layer "F.SilkS")
@@
 		)
 	)
-	(gr_text "PW1,3"
+	(gr_text "PW2,4"
 		(at 98 52 0)
 		(layer "F.SilkS")
@@
 		)
 	)
-	(gr_text "PWM0,1"
+	(gr_text "PWM1,2"
 		(at 114.6 44.2 0)
 		(layer "F.SilkS" knockout)
@@
 		)
 	)
-	(gr_text "PWM2,3"
+	(gr_text "PWM3.4"
 		(at 114.6 54.7 0)
 		(layer "F.SilkS" knockout)
@@
 	)
 	(segment
-		(start 106.362 41.656)
-		(end 101.092 41.656)
-		(width 0.25)
-		(layer "B.Cu")
-		(net "/PWM1")
-	)
-	(segment
-		(start 89.41072 53.33728)
-		(end 84.83232 53.33728)
-		(width 0.25)
-		(layer "B.Cu")
-		(net "/PWM1")
-	)
-	(segment
-		(start 101.092 41.656)
-		(end 89.41072 53.33728)
-		(width 0.25)
-		(layer "B.Cu")
-		(net "/PWM1")
-	)
-	(segment
-		(start 106.426 41.592)
-		(end 106.362 41.656)
-		(width 0.25)
-		(layer "B.Cu")
-		(net "/PWM1")
-	)
-	(segment
 		(start 106.426 37.592)
 		(end 103.952991 37.592)
 		(width 0.25)
 		(layer "B.Cu")
-		(net "/PWM0")
+		(net "/PWM1")
 	)
 	(segment
@@
 		(width 0.25)
 		(layer "B.Cu")
-		(net "/PWM0")
+		(net "/PWM1")
 	)
 	(segment
@@
 		(width 0.25)
 		(layer "B.Cu")
-		(net "/PWM0")
+		(net "/PWM1")
 	)
 	(segment
@@
 	)
 	(segment
-		(start 96.688 48.092)
-		(end 86.36272 58.41728)
+		(start 106.362 41.656)
+		(end 101.092 41.656)
 		(width 0.25)
 		(layer "B.Cu")
@@
 	)
 	(segment
-		(start 86.36272 58.41728)
-		(end 84.83232 58.41728)
+		(start 89.41072 53.33728)
+		(end 84.83232 53.33728)
 		(width 0.25)
 		(layer "B.Cu")
@@
 	)
 	(segment
-		(start 106.426 48.092)
-		(end 96.688 48.092)
+		(start 101.092 41.656)
+		(end 89.41072 53.33728)
 		(width 0.25)
 		(layer "B.Cu")
@@
 	)
 	(segment
-		(start 108.059 50.709)
-		(end 108.059 47.686485)
-		(width 0.25)
-		(layer "B.Cu")
-		(net "/PWM3")
-	)
-	(segment
-		(start 96.651 47.113)
-		(end 87.88672 55.87728)
-		(width 0.25)
-		(layer "B.Cu")
-		(net "/PWM3")
-	)
-	(segment
-		(start 108.059 47.686485)
-		(end 107.485515 47.113)
-		(width 0.25)
-		(layer "B.Cu")
-		(net "/PWM3")
-	)
-	(segment
-		(start 87.88672 55.87728)
-		(end 84.83232 55.87728)
+		(start 106.426 41.592)
+		(end 106.362 41.656)
 		(width 0.25)
 		(layer "B.Cu")
-		(net "/PWM3")
+		(net "/PWM2")
 	)
 	(segment
-		(start 106.676 52.092)
-		(end 108.059 50.709)
+		(start 96.688 48.092)
+		(end 86.36272 58.41728)
 		(width 0.25)
 		(layer "B.Cu")
@@
 	)
 	(segment
-		(start 106.426 52.092)
-		(end 106.676 52.092)
+		(start 86.36272 58.41728)
+		(end 84.83232 58.41728)
 		(width 0.25)
 		(layer "B.Cu")
@@
 	)
 	(segment
-		(start 107.485515 47.113)
-		(end 96.651 47.113)
+		(start 106.426 48.092)
+		(end 96.688 48.092)
 		(width 0.25)
 		(layer "B.Cu")
@@
 		(net "/CAN_TX")
 	)
+	(via
+		(at 47.498 54.356)
+		(size 0.6)
+		(drill 0.3)
+		(layers "F.Cu" "B.Cu")
+		(net "/I2C_SDA")
+	)
+	(segment
+		(start 59.43232 66.03728)
+		(end 59.17928 66.03728)
+		(width 0.25)
+		(layer "B.Cu")
+		(net "/I2C_SDA")
+	)
+	(segment
+		(start 47.458 54.396)
+		(end 47.498 54.356)
+		(width 0.25)
+		(layer "B.Cu")
+		(net "/I2C_SDA")
+	)
+	(segment
+		(start 40.894 54.396)
+		(end 47.458 54.396)
+		(width 0.25)
+		(layer "B.Cu")
+		(net "/I2C_SDA")
+	)
+	(segment
+		(start 59.17928 66.03728)
+		(end 47.498 54.356)
+		(width 0.25)
+		(layer "B.Cu")
+		(net "/I2C_SDA")
+	)
+	(segment
+		(start 47.204 59.396)
+		(end 47.498 59.69)
+		(width 0.25)
+		(layer "B.Cu")
+		(net "/I2C_SCL")
+	)
+	(segment
+		(start 58.10732 72.33228)
+		(end 58.10732 70.29932)
+		(width 0.25)
+		(layer "B.Cu")
+		(net "/I2C_SCL")
+	)
+	(segment
+		(start 59.43232 73.65728)
+		(end 58.10732 72.33228)
+		(width 0.25)
+		(layer "B.Cu")
+		(net "/I2C_SCL")
+	)
+	(segment
+		(start 58.10732 70.29932)
+		(end 47.498 59.69)
+		(width 0.25)
+		(layer "B.Cu")
+		(net "/I2C_SCL")
+	)
+	(segment
+		(start 40.894 59.396)
+		(end 47.204 59.396)
+		(width 0.25)
+		(layer "B.Cu")
+		(net "/I2C_SCL")
+	)
 	(segment
 		(start 41.402 72.50537)
@@
 	)
 	(segment
-		(start 36.83 68.834)
-		(end 41.402 68.834)
-		(width 0.25)
-		(layer "B.Cu")
-		(net "Net-(J9-Pin_1)")
-	)
-	(segment
-		(start 45.72 71.628)
-		(end 45.72 68.834)
-		(width 0.25)
-		(layer "B.Cu")
-		(net "Net-(J9-Pin_1)")
-	)
-	(segment
-		(start 41.402 68.834)
-		(end 45.72 68.834)
-		(width 0.25)
-		(layer "B.Cu")
-		(net "Net-(J9-Pin_1)")
-	)
-	(segment
-		(start 48.26 49.784)
-		(end 52.07 49.784)
-		(width 0.25)
-		(layer "B.Cu")
-		(net "Net-(J5-Pin_1)")
-	)
-	(segment
 		(start 48.26 41.656)
 		(end 46.99 40.386)
@@
 		(net "/CAN1-")
 	)
-	(via
-		(at 47.498 54.356)
-		(size 0.6)
-		(drill 0.3)
-		(layers "F.Cu" "B.Cu")
-		(net "/I2C_SDA")
+	(segment
+		(start 36.83 68.834)
+		(end 41.402 68.834)
+		(width 0.25)
+		(layer "B.Cu")
+		(net "Net-(J9-Pin_1)")
 	)
 	(segment
-		(start 59.43232 66.03728)
-		(end 59.17928 66.03728)
+		(start 45.72 71.628)
+		(end 45.72 68.834)
 		(width 0.25)
 		(layer "B.Cu")
-		(net "/I2C_SDA")
+		(net "Net-(J9-Pin_1)")
 	)
 	(segment
-		(start 47.458 54.396)
-		(end 47.498 54.356)
+		(start 41.402 68.834)
+		(end 45.72 68.834)
 		(width 0.25)
 		(layer "B.Cu")
-		(net "/I2C_SDA")
+		(net "Net-(J9-Pin_1)")
 	)
 	(segment
-		(start 40.894 54.396)
-		(end 47.458 54.396)
+		(start 48.26 49.784)
+		(end 52.07 49.784)
 		(width 0.25)
 		(layer "B.Cu")
-		(net "/I2C_SDA")
+		(net "Net-(J5-Pin_1)")
 	)
 	(segment
-		(start 59.17928 66.03728)
-		(end 47.498 54.356)
+		(start 108.059 50.709)
+		(end 108.059 47.686485)
 		(width 0.25)
 		(layer "B.Cu")
-		(net "/I2C_SDA")
+		(net "/PWM4")
 	)
 	(segment
-		(start 47.204 59.396)
-		(end 47.498 59.69)
+		(start 96.651 47.113)
+		(end 87.88672 55.87728)
 		(width 0.25)
 		(layer "B.Cu")
-		(net "/I2C_SCL")
+		(net "/PWM4")
 	)
 	(segment
-		(start 58.10732 72.33228)
-		(end 58.10732 70.29932)
+		(start 108.059 47.686485)
+		(end 107.485515 47.113)
 		(width 0.25)
 		(layer "B.Cu")
-		(net "/I2C_SCL")
+		(net "/PWM4")
 	)
 	(segment
-		(start 59.43232 73.65728)
-		(end 58.10732 72.33228)
+		(start 87.88672 55.87728)
+		(end 84.83232 55.87728)
 		(width 0.25)
 		(layer "B.Cu")
-		(net "/I2C_SCL")
+		(net "/PWM4")
 	)
 	(segment
-		(start 58.10732 70.29932)
-		(end 47.498 59.69)
+		(start 106.676 52.092)
+		(end 108.059 50.709)
 		(width 0.25)
 		(layer "B.Cu")
-		(net "/I2C_SCL")
+		(net "/PWM4")
 	)
 	(segment
-		(start 40.894 59.396)
-		(end 47.204 59.396)
+		(start 106.426 52.092)
+		(end 106.676 52.092)
 		(width 0.25)
 		(layer "B.Cu")
-		(net "/I2C_SCL")
+		(net "/PWM4")
+	)
+	(segment
+		(start 107.485515 47.113)
+		(end 96.651 47.113)
+		(width 0.25)
+		(layer "B.Cu")
+		(net "/PWM4")
 	)
 	(zone

Commit message: ESP32基板　予備GPIOのシルクを修正，ver 0.5
Other:
- board text added: "BoardID: TS26-CTRL-ESP32 ver 0.5"
- board text added: "GPIO13,32,33"
- board text removed: "BoardID: TS26-CTRL-ESP32 ver 0.4"
- board text removed: "GPIO13,23, 32,33"
Changed lines of the file:
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@@
 	)
 	(gr_rect
-		(start 76.962 21.352)
-		(end 82.962 25.352)
+		(start 75.3 27.7)
+		(end 81.3 31.7)
 		(stroke
 			(width 0.15)
@@
 		(layer "F.SilkS")
 	)
+	(gr_rect
+		(start 76.5 22)
+		(end 82.5 26)
+		(stroke
+			(width 0.15)
+			(type solid)
+		)
+		(fill no)
+		(layer "F.SilkS")
+	)
 	(gr_line
-		(start 78.962 21.352)
-		(end 78.962 25.352)
+		(start 77.3 27.7)
+		(end 77.3 31.7)
 		(stroke
 			(width 0.1)
@@
 	)
 	(gr_line
-		(start 79.635 26.924)
-		(end 79.962 25.352)
-		(stroke
-			(width 0.15)
-			(type solid)
-		)
-		(layer "F.SilkS")
-	)
-	(gr_line
-		(start 80.962 21.352)
-		(end 80.962 25.352)
+		(start 78.5 22)
+		(end 78.5 26)
 		(stroke
 			(width 0.1)
@@
 	)
 	(gr_line
-		(start 85.852 29.972)
+		(start 79.3 27.7)
+		(end 79.3 31.7)
+		(stroke
+			(width 0.1)
+			(type default)
+		)
+		(layer "F.SilkS")
+	)
+	(gr_line
+		(start 80.5 22)
+		(end 80.5 26)
+		(stroke
+			(width 0.1)
+			(type default)
+		)
+		(layer "F.SilkS")
+	)
+	(gr_line
+		(start 85.9 30.4)
 		(end 87.63 31.242)
 		(stroke
@@
 		)
 	)
-	(gr_text "GPIO13,23,\n	32,33"
-		(at 75.184 26.924 0)
-		(layer "F.SilkS" knockout)
-		(effects
-			(font
-				(size 1 1)
-				(thickness 0.2)
-				(bold yes)
-			)
-			(justify left top)
-		)
-	)
 	(gr_text "Lp-C  ローパスフィルタ用C,\nP-dn  もしくはプルダウン"
 		(at 87.5 72 0)
@@
 		)
 	)
-	(gr_text "BoardID:\n TS26-CTRL-ESP32\n\nver 0.4"
+	(gr_text "BoardID:\n TS26-CTRL-ESP32\n\nver 0.5"
 		(at 39 24.5 0)
 		(layer "F.SilkS")
@@
 		)
 	)
+	(gr_text "GPIO13,32,33"
+		(at 75.1 27.5 0)
+		(layer "F.SilkS" knockout)
+		(effects
+			(font
+				(size 1 1)
+				(thickness 0.2)
+				(bold yes)
+			)
+			(justify left bottom)
+		)
+	)
+	(gr_text "GPIO23"
+		(at 76.3 21.9 0)
+		(layer "F.SilkS" knockout)
+		(effects
+			(font
+				(size 1 1)
+				(thickness 0.2)
+				(bold yes)
+			)
+			(justify left bottom)
+		)
+	)
 	(gr_text "IO"
 		(at 41.402 74.168 0)
@@
 		)
 	)
+	(gr_text "IO"
+		(at 76.3 28 90)
+		(layer "F.SilkS")
+		(effects
+			(font
+				(size 1 1)
+				(thickness 0.2)
+				(bold yes)
+			)
+			(justify right)
+		)
+	)
 	(gr_text "GND"
-		(at 77.962 21.652 90)
+		(at 77.5 22.3 90)
 		(layer "F.SilkS")
 		(effects
@@
 	)
 	(gr_text "3.3V"
-		(at 79.962 21.652 90)
+		(at 78.3 28 90)
 		(layer "F.SilkS")
 		(effects
@@
 		)
 	)
+	(gr_text "3.3V"
+		(at 79.5 22.3 90)
+		(layer "F.SilkS")
+		(effects
+			(font
+				(size 1 1)
+				(thickness 0.2)
+				(bold yes)
+			)
+			(justify right)
+		)
+	)
+	(gr_text "GND"
+		(at 80.3 28.2 90)
+		(layer "F.SilkS")
+		(effects
+			(font
+				(size 1 1)
+				(thickness 0.2)
+				(bold yes)
+			)
+			(justify right)
+		)
+	)
 	(gr_text "IO"
-		(at 81.962 21.652 90)
+		(at 81.5 22.3 90)
 		(layer "F.SilkS")
 		(effects
@@
 	)
 	(gr_text "5V"
-		(at 85.852 27.94 180)
+		(at 85.852 28.5 180)
 		(layer "F.SilkS" knockout)
 		(effects
@@
 	)
 	(segment
+		(start 106.362 41.656)
+		(end 101.092 41.656)
+		(width 0.25)
+		(layer "B.Cu")
+		(net "/PWM2")
+	)
+	(segment
+		(start 89.41072 53.33728)
+		(end 84.83232 53.33728)
+		(width 0.25)
+		(layer "B.Cu")
+		(net "/PWM2")
+	)
+	(segment
+		(start 101.092 41.656)
+		(end 89.41072 53.33728)
+		(width 0.25)
+		(layer "B.Cu")
+		(net "/PWM2")
+	)
+	(segment
+		(start 106.426 41.592)
+		(end 106.362 41.656)
+		(width 0.25)
+		(layer "B.Cu")
+		(net "/PWM2")
+	)
+	(segment
 		(start 106.426 37.592)
 		(end 103.952991 37.592)
@@
 	)
 	(segment
-		(start 106.362 41.656)
-		(end 101.092 41.656)
-		(width 0.25)
-		(layer "B.Cu")
-		(net "/PWM2")
-	)
-	(segment
-		(start 89.41072 53.33728)
-		(end 84.83232 53.33728)
-		(width 0.25)
-		(layer "B.Cu")
-		(net "/PWM2")
-	)
-	(segment
-		(start 101.092 41.656)
-		(end 89.41072 53.33728)
-		(width 0.25)
-		(layer "B.Cu")
-		(net "/PWM2")
-	)
-	(segment
-		(start 106.426 41.592)
-		(end 106.362 41.656)
-		(width 0.25)
-		(layer "B.Cu")
-		(net "/PWM2")
-	)
-	(segment
 		(start 96.688 48.092)
 		(end 86.36272 58.41728)
@@
 		(layer "B.Cu")
 		(net "/PWM3")
+	)
+	(segment
+		(start 108.059 50.709)
+		(end 108.059 47.686485)
+		(width 0.25)
+		(layer "B.Cu")
+		(net "/PWM4")
+	)
+	(segment
+		(start 96.651 47.113)
+		(end 87.88672 55.87728)
+		(width 0.25)
+		(layer "B.Cu")
+		(net "/PWM4")
+	)
+	(segment
+		(start 108.059 47.686485)
+		(end 107.485515 47.113)
+		(width 0.25)
+		(layer "B.Cu")
+		(net "/PWM4")
+	)
+	(segment
+		(start 87.88672 55.87728)
+		(end 84.83232 55.87728)
+		(width 0.25)
+		(layer "B.Cu")
+		(net "/PWM4")
+	)
+	(segment
+		(start 106.676 52.092)
+		(end 108.059 50.709)
+		(width 0.25)
+		(layer "B.Cu")
+		(net "/PWM4")
+	)
+	(segment
+		(start 106.426 52.092)
+		(end 106.676 52.092)
+		(width 0.25)
+		(layer "B.Cu")
+		(net "/PWM4")
+	)
+	(segment
+		(start 107.485515 47.113)
+		(end 96.651 47.113)
+		(width 0.25)
+		(layer "B.Cu")
+		(net "/PWM4")
 	)
 	(segment
@@
 		(net "Net-(J5-Pin_1)")
 	)
-	(segment
-		(start 108.059 50.709)
-		(end 108.059 47.686485)
-		(width 0.25)
-		(layer "B.Cu")
-		(net "/PWM4")
-	)
-	(segment
-		(start 96.651 47.113)
-		(end 87.88672 55.87728)
-		(width 0.25)
-		(layer "B.Cu")
-		(net "/PWM4")
-	)
-	(segment
-		(start 108.059 47.686485)
-		(end 107.485515 47.113)
-		(width 0.25)
-		(layer "B.Cu")
-		(net "/PWM4")
-	)
-	(segment
-		(start 87.88672 55.87728)
-		(end 84.83232 55.87728)
-		(width 0.25)
-		(layer "B.Cu")
-		(net "/PWM4")
-	)
-	(segment
-		(start 106.676 52.092)
-		(end 108.059 50.709)
-		(width 0.25)
-		(layer "B.Cu")
-		(net "/PWM4")
-	)
-	(segment
-		(start 106.426 52.092)
-		(end 106.676 52.092)
-		(width 0.25)
-		(layer "B.Cu")
-		(net "/PWM4")
-	)
-	(segment
-		(start 107.485515 47.113)
-		(end 96.651 47.113)
-		(width 0.25)
-		(layer "B.Cu")
-		(net "/PWM4")
-	)
 	(zone
