File: ESP32-DevKitC_control_board/ESP32-DevKitC_control_board.kicad_pcb (KiCad board)
At the start: 2 copper layers, 85 x 60 mm, 39 parts, among them J1 Conn_01x02_Pin, J10 Conn_01x03_Pin, J11 Conn_01x03_Pin, J2 Conn_01x03_Pin, J3 Conn_01x03_Pin, J4 Conn_01x02_Pin, J5 Conn_01x02_Pin, J6 Conn_01x02_Pin, J7 Conn_01x04_Pin, J8 Conn_01x03_Pin, J9 Conn_01x03_Pin, U1 MCP2562-E-P, U2 ESP32-DevKitC

Commit message: ESP32基板　シルクを一部修正，3Dモデルを追加，ver 1.0
Parts:
- renumbered C2 to C1, C1 to C2, D4 to D1, J2 to J1, J3 to J2, J1 to J3, J5 to J4, J4 to J5, J7 to J6, J6 to J7, R12 to R1, R9 to R10, R10 to R11, R11 to R12, R1 to R2, R2 to R3, R3 to R4, R4 to R5, R5 to R6, R6 to R7, R7 to R8, R8 to R9
Routing:
- net /I2C_SDA: vias 1 -> 0
Other:
- board text added: "2026/10/10 Designed by E.Yoshioka"
- board text added: "BoardID: TS26-CTRL-ESP32 ver 1.0"
- board text removed: "2026/10/02 Designed by E.Yoshioka"
- board text removed: "BoardID: TS26-CTRL-ESP32 ver 0.5"
Changed lines of the file:
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@@
 		(descr "C, Disc series, Radial, pin pitch=2.50mm, diameter*width=5*2.5mm^2, Capacitor, http://cdn-reichelt.de/documents/datenblatt/B300/DS_KERKO_TC.pdf")
 		(tags "C Disc series Radial pin pitch 2.50mm diameter 5mm width 2.5mm Capacitor")
-		(property "Reference" "C2"
+		(property "Reference" "C1"
 			(at 4.786 -1.27 0)
 			(layer "F.SilkS")
@@
 		(at 106.426 39.592 -90)
 		(descr "Header 3 pin, side entry type, 2mm pitch.")
-		(property "Reference" "J2"
+		(property "Reference" "J1"
 			(at -5.092 1.426 180)
 			(layer "F.SilkS")
@@
 		(descr "Hirose DF1E series connector, 2 pins, right-angle, pitch 2.50mm")
 		(tags "connector Hirose DF1E right-angle 2pin 2.5mm")
-		(property "Reference" "J6"
+		(property "Reference" "J7"
 			(at -4.012 2.606 180)
 			(layer "F.SilkS")
@@
 		)
 		(embedded_fonts no)
+		(model "${KIPRJMOD}/../common_lib/3dmodels/ESP32-DEVKITC-32D--3DModel-STEP-269445.STEP"
+			(offset
+				(xyz 12.7 -19.75 9)
+			)
+			(scale
+				(xyz 1 1 1)
+			)
+			(rotate
+				(xyz -90 -0 -0)
+			)
+		)
 	)
 	(footprint "Resistor_THT:R_Axial_DIN0207_L6.3mm_D2.5mm_P2.54mm_Vertical"
@@
 		(descr "Resistor, Axial_DIN0207 series, Axial, Vertical, pin pitch=2.54mm, 0.25W = 1/4W, length*diameter=6.3*2.5mm^2, http://cdn-reichelt.de/documents/datenblatt/B400/1_4W%23YAG.pdf")
 		(tags "Resistor Axial_DIN0207 series Axial Vertical pin pitch 2.54mm 0.25W = 1/4W length 6.3mm diameter 2.5mm")
-		(property "Reference" "R7"
+		(property "Reference" "R8"
 			(at -2.794 0 90)
 			(layer "F.SilkS")
@@
 		(descr "Resistor, Axial_DIN0207 series, Axial, Vertical, pin pitch=2.54mm, 0.25W = 1/4W, length*diameter=6.3*2.5mm^2, http://cdn-reichelt.de/documents/datenblatt/B400/1_4W%23YAG.pdf")
 		(tags "Resistor Axial_DIN0207 series Axial Vertical pin pitch 2.54mm 0.25W = 1/4W length 6.3mm diameter 2.5mm")
-		(property "Reference" "R12"
+		(property "Reference" "R1"
 			(at -2.46 0 0)
 			(layer "F.SilkS")
@@
 			(layers "*.Cu" "*.Mask")
 			(remove_unused_layers no)
-			(net "Net-(D4-A)")
+			(net "Net-(D1-A)")
 			(pintype "passive")
 		)
@@
 		(descr "Resistor, Axial_DIN0207 series, Axial, Vertical, pin pitch=2.54mm, 0.25W = 1/4W, length*diameter=6.3*2.5mm^2, http://cdn-reichelt.de/documents/datenblatt/B400/1_4W%23YAG.pdf")
 		(tags "Resistor Axial_DIN0207 series Axial Vertical pin pitch 2.54mm 0.25W = 1/4W length 6.3mm diameter 2.5mm")
-		(property "Reference" "R11"
+		(property "Reference" "R12"
 			(at 4.476 0 180)
 			(layer "F.SilkS")
@@
 		(at 106.426 50.092 -90)
 		(descr "Header 3 pin, side entry type, 2mm pitch.")
-		(property "Reference" "J3"
+		(property "Reference" "J2"
 			(at -5.092 2.926 180)
 			(layer "F.SilkS")
@@
 		(descr "Hirose DF1E series connector, 4 pins, right-angle, pitch 2.50mm")
 		(tags "connector Hirose DF1E right-angle 4pin 2.5mm")
-		(property "Reference" "J7"
+		(property "Reference" "J6"
 			(at 9.196 4.606 180)
 			(layer "F.SilkS")
@@
 		(descr "Hirose DF1E series connector, 2 pins, right-angle, pitch 2.50mm")
 		(tags "connector Hirose DF1E right-angle 2pin 2.5mm")
-		(property "Reference" "J4"
+		(property "Reference" "J5"
 			(at -1.836 4.406 180)
 			(layer "F.SilkS")
@@
 		(descr "LED, diameter 5.0mm, 2 pins, http://cdn-reichelt.de/documents/datenblatt/A500/LL-504BC2E-009.pdf, generated by kicad-footprint-generator")
 		(tags "LED")
-		(property "Reference" "D4"
+		(property "Reference" "D1"
 			(at -1.46 3.25 90)
 			(layer "F.SilkS")
@@
 			(layers "*.Cu" "*.Mask")
 			(remove_unused_layers no)
-			(net "Net-(D4-A)")
+			(net "Net-(D1-A)")
 			(pinfunction "A_2")
 			(pintype "passive")
@@
 		(descr "Resistor, Axial_DIN0207 series, Axial, Vertical, pin pitch=2.54mm, 0.25W = 1/4W, length*diameter=6.3*2.5mm^2, http://cdn-reichelt.de/documents/datenblatt/B400/1_4W%23YAG.pdf")
 		(tags "Resistor Axial_DIN0207 series Axial Vertical pin pitch 2.54mm 0.25W = 1/4W length 6.3mm diameter 2.5mm")
-		(property "Reference" "R10"
+		(property "Reference" "R11"
 			(at 4.612 0 180)
 			(layer "F.SilkS")
@@
 		(descr "Hirose DF1E series connector, 2 pins, right-angle, pitch 2.50mm")
 		(tags "connector Hirose DF1E right-angle 2pin 2.5mm")
-		(property "Reference" "J1"
+		(property "Reference" "J3"
 			(at 6.17 1.254 90)
 			(layer "F.SilkS")
@@
 		(descr "Resistor, Axial_DIN0207 series, Axial, Vertical, pin pitch=2.54mm, 0.25W = 1/4W, length*diameter=6.3*2.5mm^2, http://cdn-reichelt.de/documents/datenblatt/B400/1_4W%23YAG.pdf")
 		(tags "Resistor Axial_DIN0207 series Axial Vertical pin pitch 2.54mm 0.25W = 1/4W length 6.3mm diameter 2.5mm")
-		(property "Reference" "R3"
+		(property "Reference" "R4"
 			(at 0.596 2.502 90)
 			(layer "F.SilkS")
@@
 		(descr "Through hole straight pin header, 1x02, 2.54mm pitch, single row")
 		(tags "Through hole pin header THT 1x02 2.54mm single row")
-		(property "Reference" "J5"
+		(property "Reference" "J4"
 			(at 0 -2.54 0)
 			(layer "F.SilkS")
@@
 			(layers "*.Cu" "*.Mask")
 			(remove_unused_layers no)
-			(net "Net-(J5-Pin_1)")
+			(net "Net-(J4-Pin_1)")
 			(pinfunction "Pin_1_1")
 			(pintype "passive")
@@
 		(descr "Resistor, Axial_DIN0207 series, Axial, Vertical, pin pitch=2.54mm, 0.25W = 1/4W, length*diameter=6.3*2.5mm^2, http://cdn-reichelt.de/documents/datenblatt/B400/1_4W%23YAG.pdf")
 		(tags "Resistor Axial_DIN0207 series Axial Vertical pin pitch 2.54mm 0.25W = 1/4W length 6.3mm diameter 2.5mm")
-		(property "Reference" "R9"
+		(property "Reference" "R10"
 			(at 1.016 2.032 270)
 			(layer "F.SilkS")
@@
 		(descr "Resistor, Axial_DIN0207 series, Axial, Vertical, pin pitch=2.54mm, 0.25W = 1/4W, length*diameter=6.3*2.5mm^2, http://cdn-reichelt.de/documents/datenblatt/B400/1_4W%23YAG.pdf")
 		(tags "Resistor Axial_DIN0207 series Axial Vertical pin pitch 2.54mm 0.25W = 1/4W length 6.3mm diameter 2.5mm")
-		(property "Reference" "R6"
+		(property "Reference" "R7"
 			(at -1.27 2.032 90)
 			(layer "F.SilkS")
@@
 		(descr "Resistor, Axial_DIN0207 series, Axial, Vertical, pin pitch=2.54mm, 0.25W = 1/4W, length*diameter=6.3*2.5mm^2, http://cdn-reichelt.de/documents/datenblatt/B400/1_4W%23YAG.pdf")
 		(tags "Resistor Axial_DIN0207 series Axial Vertical pin pitch 2.54mm 0.25W = 1/4W length 6.3mm diameter 2.5mm")
-		(property "Reference" "R5"
+		(property "Reference" "R6"
 			(at 0.508 2.54 90)
 			(layer "F.SilkS")
@@
 		(descr "Resistor, Axial_DIN0207 series, Axial, Vertical, pin pitch=2.54mm, 0.25W = 1/4W, length*diameter=6.3*2.5mm^2, http://cdn-reichelt.de/documents/datenblatt/B400/1_4W%23YAG.pdf")
 		(tags "Resistor Axial_DIN0207 series Axial Vertical pin pitch 2.54mm 0.25W = 1/4W length 6.3mm diameter 2.5mm")
-		(property "Reference" "R2"
+		(property "Reference" "R3"
 			(at 0.596 2.502 90)
 			(layer "F.SilkS")
@@
 		(descr "Resistor, Axial_DIN0207 series, Axial, Vertical, pin pitch=2.54mm, 0.25W = 1/4W, length*diameter=6.3*2.5mm^2, http://cdn-reichelt.de/documents/datenblatt/B400/1_4W%23YAG.pdf")
 		(tags "Resistor Axial_DIN0207 series Axial Vertical pin pitch 2.54mm 0.25W = 1/4W length 6.3mm diameter 2.5mm")
-		(property "Reference" "R4"
+		(property "Reference" "R5"
 			(at -2.124 0.012 180)
 			(layer "F.SilkS")
@@
 		(descr "CP, Radial series, Radial, pin pitch=2.50mm, diameter=6.3mm, height=7mm, Electrolytic Capacitor")
 		(tags "CP Radial series Radial pin pitch 2.50mm diameter 6.3mm height 7mm Electrolytic Capacitor")
-		(property "Reference" "C1"
+		(property "Reference" "C2"
 			(at 4.826 -2.54 180)
 			(layer "F.SilkS")
@@
 		(descr "Resistor, Axial_DIN0207 series, Axial, Vertical, pin pitch=2.54mm, 0.25W = 1/4W, length*diameter=6.3*2.5mm^2, http://cdn-reichelt.de/documents/datenblatt/B400/1_4W%23YAG.pdf")
 		(tags "Resistor Axial_DIN0207 series Axial Vertical pin pitch 2.54mm 0.25W = 1/4W length 6.3mm diameter 2.5mm")
-		(property "Reference" "R8"
+		(property "Reference" "R9"
 			(at 4.416 0.33 180)
 			(layer "F.SilkS")
@@
 		(descr "Resistor, Axial_DIN0207 series, Axial, Vertical, pin pitch=2.54mm, 0.25W = 1/4W, length*diameter=6.3*2.5mm^2, http://cdn-reichelt.de/documents/datenblatt/B400/1_4W%23YAG.pdf")
 		(tags "Resistor Axial_DIN0207 series Axial Vertical pin pitch 2.54mm 0.25W = 1/4W length 6.3mm diameter 2.5mm")
-		(property "Reference" "R1"
+		(property "Reference" "R2"
 			(at -2.54 0 180)
 			(layer "F.SilkS")
@@
 			(layers "*.Cu" "*.Mask")
 			(remove_unused_layers no)
-			(net "Net-(J5-Pin_1)")
+			(net "Net-(J4-Pin_1)")
 			(pintype "passive")
 		)
@@
 		)
 	)
-	(gr_text "BoardID:\n TS26-CTRL-ESP32\n\nver 0.5"
+	(gr_text "BoardID:\n TS26-CTRL-ESP32\n\nver 1.0"
 		(at 39 24.5 0)
 		(layer "F.SilkS")
@@
 		)
 	)
-	(gr_text "2026/10/02\nDesigned by E.Yoshioka"
+	(gr_text "2026/10/10\nDesigned by E.Yoshioka"
 		(at 66.04 23.876 0)
 		(layer "B.SilkS")
@@
 		(net "/CAN_TX")
 	)
-	(via
-		(at 47.498 54.356)
-		(size 0.6)
-		(drill 0.3)
-		(layers "F.Cu" "B.Cu")
-		(net "/I2C_SDA")
-	)
 	(segment
 		(start 59.43232 66.03728)
@@
 		(width 0.25)
 		(layer "F.Cu")
-		(net "Net-(D4-A)")
+		(net "Net-(D1-A)")
 	)
 	(segment
@@
 		(width 0.25)
 		(layer "F.Cu")
-		(net "Net-(D4-A)")
+		(net "Net-(D1-A)")
 	)
 	(segment
@@
 		(width 0.25)
 		(layer "B.Cu")
-		(net "Net-(J5-Pin_1)")
+		(net "Net-(J4-Pin_1)")
 	)
 	(zone

Commit message: ESP32基板　QRを追加，ver 1.1
Routing:
- net GND: vias 122 -> 120
Other:
- board text added: "BoardID: TS26-CTRL-ESP32 ver 1.1"
- board text removed: "BoardID: TS26-CTRL-ESP32 ver 1.0"
Changed lines of the file:
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@@
+	)
+	(gr_rect
+		(start 68.5 46)
+		(end 76.5 54)
+		(stroke
+			(width 0)
+			(type solid)
+		)
+		(fill yes)
+		(layer "B.SilkS")
 	)
 	(gr_rect
@@
 		)
 	)
-	(gr_text "BoardID:\n TS26-CTRL-ESP32\n\nver 1.0"
+	(gr_text "BoardID:\n TS26-CTRL-ESP32\n\nver 1.1"
 		(at 39 24.5 0)
 		(layer "F.SilkS")
@@
 	)
 	(via
-		(at 70 50)
-		(size 0.8)
-		(drill 0.4)
-		(layers "F.Cu" "B.Cu")
-		(free yes)
-		(net "GND")
-	)
-	(via
 		(at 35 38)
 		(size 0.8)
@@
 		(size 0.8)
 		(drill 0.4)
-		(layers "F.Cu" "B.Cu")
-		(free yes)
-		(net "GND")
-	)
-	(via
-		(at 75 50)
-		(size 0.8)
-		(drill 0.4)
