File: DCmotor_control_board/DCmotor_control_board.kicad_pcb (KiCad board)
At the start: 2 copper layers, 45 x 55 mm, 31 parts, among them J1 Conn_01x02_Pin, J2 Conn_01x04_Pin, J3 Conn_01x02_Pin, J4 Conn_01x04_Pin, J5 Conn_01x02_Pin, U1 L7805CV, U2 TLP2745, U3 TLP2745, U4 TB67H450FNG_EL, U5 TLP2745, U6 TLP2745, U7 TB67H450FNG_EL

Commit message: モータドライバ基板　シルクを一部修正，ver 1.0
Parts:
- renumbered J4 to J3, J3 to J4
Other:
- board text added: "2026/10/10 Designed by E.Yoshioka"
- board text added: "POWER"
- board text added: "ver 1.0"
- board text removed: "2026/10/03 Designed by E.Yoshioka"
- board text removed: "DRIVE"
- board text removed: "ver 0.1"
Changed lines of the file:
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@@
 			)
 		)
+		(property "Buy_URL" "https://akizukidenshi.com/catalog/g/g118360/"
+			(at 0 0 270)
+			(unlocked yes)
+			(layer "F.Fab")
+			(hide yes)
+			(effects
+				(font
+					(size 1 1)
+					(thickness 0.15)
+				)
+			)
+		)
 		(property ki_fp_filters "SO*6L*10x3.84mm*P1.27mm*")
 		(sheetname "/")
@@
 			)
 		)
+		(property "Buy_URL" "https://akizukidenshi.com/catalog/g/g118360/"
+			(at 0 0 270)
+			(unlocked yes)
+			(layer "F.Fab")
+			(hide yes)
+			(effects
+				(font
+					(size 1 1)
+					(thickness 0.15)
+				)
+			)
+		)
 		(property ki_fp_filters "SO*6L*10x3.84mm*P1.27mm*")
 		(sheetname "/")
@@
 			)
 		)
+		(property "Buy_URL" "https://akizukidenshi.com/catalog/g/g118360/"
+			(at 0 0 270)
+			(unlocked yes)
+			(layer "F.Fab")
+			(hide yes)
+			(effects
+				(font
+					(size 1 1)
+					(thickness 0.15)
+				)
+			)
+		)
 		(property ki_fp_filters "SO*6L*10x3.84mm*P1.27mm*")
 		(sheetname "/")
@@
 		(descr "Hirose DF1E series connector, 4 pins, right-angle, pitch 2.50mm")
 		(tags "connector Hirose DF1E right-angle 4pin 2.5mm")
-		(property "Reference" "J4"
+		(property "Reference" "J3"
 			(at -1.898 4.572 180)
 			(layer "F.SilkS")
@@
 			(layers "*.Cu" "*.Mask")
 			(remove_unused_layers no)
-			(net "unconnected-(J4-Pin_3-Pad3)")
+			(net "unconnected-(J3-Pin_3-Pad3)")
 			(pinfunction "Pin_3_3")
 			(pintype "passive+no_connect")
@@
 			)
 		)
+		(property "Buy_URL" "https://akizukidenshi.com/catalog/g/g118360/"
+			(at 0 0 270)
+			(unlocked yes)
+			(layer "F.Fab")
+			(hide yes)
+			(effects
+				(font
+					(size 1 1)
+					(thickness 0.15)
+				)
+			)
+		)
 		(property ki_fp_filters "SO*6L*10x3.84mm*P1.27mm*")
 		(sheetname "/")
@@
 		(descr "Hirose DF1E series connector, 2 pins, right-angle, pitch 2.50mm")
 		(tags "connector Hirose DF1E right-angle 2pin 2.5mm")
-		(property "Reference" "J3"
+		(property "Reference" "J4"
 			(at 6.35 -9.906 180)
 			(layer "F.SilkS")
@@
 			(remove_unused_layers no)
 			(roundrect_rratio 0.25)
-			(net "Net-(J3-Pin_1)")
+			(net "Net-(J4-Pin_1)")
 			(pinfunction "Pin_1_1")
 			(pintype "passive")
@@
 			(layers "*.Cu" "*.Mask")
 			(remove_unused_layers no)
-			(net "Net-(J3-Pin_2)")
+			(net "Net-(J4-Pin_2)")
 			(pinfunction "Pin_2_2")
 			(pintype "passive")
@@
 			(size 1.202401 0.42)
 			(layers "B.Cu" "B.Mask" "B.Paste")
-			(net "Net-(J3-Pin_1)")
+			(net "Net-(J4-Pin_1)")
 			(pinfunction "OUT1_6")
 			(pintype "output")
@@
 			(size 1.202401 0.42)
 			(layers "B.Cu" "B.Mask" "B.Paste")
-			(net "Net-(J3-Pin_2)")
+			(net "Net-(J4-Pin_2)")
 			(pinfunction "OUT2_8")
 			(pintype "output")
@@
 		(layer "Edge.Cuts")
 	)
-	(gr_text "DRIVE"
+	(gr_text "POWER"
 		(at 36.83 53.086 0)
 		(layer "F.SilkS" knockout)
@@
 		)
 	)
-	(gr_text "ver 0.1"
+	(gr_text "ver 1.0"
 		(at 68 64 0)
 		(layer "F.SilkS")
@@
 		)
 	)
-	(gr_text "2026/10/03\nDesigned by\nE.Yoshioka"
+	(gr_text "2026/10/10\nDesigned by\nE.Yoshioka"
 		(at 38.862 74.93 270)
 		(layer "B.SilkS")
@@
 		(width 0.8)
 		(layer "B.Cu")
-		(net "Net-(J3-Pin_1)")
+		(net "Net-(J4-Pin_1)")
 	)
 	(segment
@@
 		(width 0.8)
 		(layer "B.Cu")
-		(net "Net-(J3-Pin_2)")
+		(net "Net-(J4-Pin_2)")
 	)
 	(segment
@@
 		(width 0.8)
 		(layer "B.Cu")
-		(net "Net-(J3-Pin_2)")
+		(net "Net-(J4-Pin_2)")
 	)
 	(zone

Commit message: モータドライバ基板　シリアルコード用QRを追加，ver 1.1
Other:
- board text added: "ver 1.1"
- board text removed: "ver 1.0"
Changed lines of the file:
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@@
+	)
+	(gr_rect
+		(start 42.712 73.954)
+		(end 47.712 78.954)
+		(stroke
+			(width 0)
+			(type solid)
+		)
+		(fill yes)
+		(layer "B.SilkS")
 	)
 	(gr_rect
@@
 		)
 	)
-	(gr_text "ver 1.0"
+	(gr_text "ver 1.1"
 		(at 68 64 0)
 		(layer "F.SilkS")
