File: Nucleo-F446RE_control_board/Nucleo-F446RE_control_board.kicad_pcb (KiCad board)
At the start: 2 copper layers, 100 x 90 mm, 51 parts, among them J1 Conn_01x02_Pin, J10 Conn_01x03_Pin, J11 Conn_01x03_Pin, J12 Conn_01x03_Pin, J13 Conn_01x04_Pin, J14 Conn_01x04_Pin, J15 Conn_01x02_Pin, J16 Conn_01x02_Pin, J2 Conn_01x03_Pin, J3 Conn_01x03_Pin, J4 Conn_01x03_Pin, J5 Conn_01x03_Pin, J6 Conn_01x03_Pin, J7 Conn_01x02_Pin, J8 Conn_01x02_Pin, J9 Conn_01x04_Pin, U2 MCP2562-E-P, U3 MCP2562-E-P

Commit message: F446RE基板　シルクを一部修正，ver 1.0
Routing:
- net GND: vias 228 -> 227
Other:
- board text added: "2026/10/10 Designed by E.Yoshioka"
- board text added: "BoardID: TS26-CTRL-F446RE ver 1.0"
- board text removed: "2026/10/03 Designed by E.Yoshioka"
- board text removed: "BoardID: TS26-CTRL-F446RE ver 0.5"
Changed lines of the file:
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@@
 			)
 			(scale
-				(xyz 1 1 1)
+				(xyz 1 1 1.746031746)
 			)
 			(rotate
-				(xyz 0 0 0)
+				(xyz -0 -0 -0)
 			)
 		)
@@
 	)
 	(gr_rect
+		(start 51.054 72.01)
+		(end 59.054 80.01)
+		(stroke
+			(width 0)
+			(type solid)
+		)
+		(fill yes)
+		(layer "B.SilkS")
+	)
+	(gr_rect
 		(start 56.588 102.828)
 		(end 69.088 109.728)
@@
 		)
 	)
-	(gr_text "BoardID:\n TS26-CTRL-F446RE\n\nver 0.5"
+	(gr_text "BoardID:\n TS26-CTRL-F446RE\n\nver 1.0"
 		(at 45.974 107.696 0)
 		(layer "F.SilkS")
@@
 		)
 	)
-	(gr_text "2026/10/03\nDesigned by E.Yoshioka"
+	(gr_text "2026/10/10\nDesigned by E.Yoshioka"
 		(at 74.168 94.742 0)
 		(layer "B.SilkS")
@@
 	)
 	(via
-		(at 55 76)
-		(size 0.8)
-		(drill 0.4)
-		(layers "F.Cu" "B.Cu")
-		(free yes)
-		(net "GND")
-	)
-	(via
