File: Nucleo-F446RE_control_board/Nucleo-F446RE_control_board.kicad_sch (KiCad schematic)
At the start: 45 parts, among them J1 Conn_01x02_Pin, J10 Conn_01x03_Pin, J11 Conn_01x03_Pin, J12 Conn_01x03_Pin, J13 Conn_01x02_Pin, J14 Conn_01x02_Pin, J15 Conn_01x03_Pin, J16 Conn_01x04_Pin, J2 Conn_01x03_Pin, J3 Conn_01x03_Pin, J4 Conn_01x02_Pin, J5 Conn_01x02_Pin, J6 Conn_01x02_Pin, J7 Conn_01x04_Pin, J8 Conn_01x03_Pin, J9 Conn_01x03_Pin, U1 NUCLEO-F446RE, U2 MCP2562-E-P, U3 MCP2562-E-P

Commit message: F446RE基板　基板完成，ver0.1
Parts:
- removed U1: NUCLEO-F446RE, OU_Micon:F446RE_mainPIN, symbol OU_Micon:NUCLEO-F446RE
- added U1: (no value), OU_Micon:F446RE_mainPIN, symbol OU_Micon:F446RE_mainPIN
- renumbered C8 to C10, C4 to C3, C5 to C4, C6 to C5, C7 to C6, C10 to C7, C3 to C8, D4 to D1, J2 to J10, J3 to J11, J16 to J13, J6 to J14, J13 to J15, J14 to J16, J8 to J2, J9 to J3, J10 to J4, J11 to J5, J15 to J6, J5 to J7, J4 to J8, J7 to J9, R15 to R1, R11 to R10, R13 to R11, R1 to R12, R2 to R13, R3 to R14, R12 to R15, R4 to R2, R5 to R3, R6 to R4, R7 to R5, R14 to R6, R8 to R7, R9 to R8, R10 to R9
Connections:
- net +3.3V: now also U1.CN7_16 (CN7_+3V3)
- net +5V: now also U1.CN7_6 (E5V)
- net CAN1_RX: now also U1.CN10_14 (PA11)
- net CAN1_TX: now also U1.CN10_12 (PA12)
- net CAN2_RX: now also U1.CN10_16 (PB12)
- net CAN2_TX: now also U1.CN10_30 (PB13)
- net GND: now also U1.CN10_20 (CN10_GND__1), U1.CN10_9 (CN10_GND), U1.CN7_19 (CN7_GND__1), U1.CN7_20 (CN7_GND__2), U1.CN7_22 (CN7_GND__3), U1.CN7_8 (CN7_GND)
- net I2C_SCL: now also U1.CN10_3 (PB8)
- net I2C_SDA: now also U1.CN10_5 (PB9)
- net PA4: now also U1.CN7_32 (PA4)
- net PA9: now also U1.CN10_21 (PA9)
- net PB0: now also U1.CN7_34 (PB0)
- net PB14: now also U1.CN10_28 (PB14)
- net PB15: now also U1.CN10_26 (PB15)
- net PC10: now also U1.CN7_1 (PC10)
- net PC2: now also U1.CN7_35 (PC2)
- net PC3: now also U1.CN7_37 (PC3)
- net PWM1: now also U1.CN10_4 (PC6)
- net PWM2: now also U1.CN10_19 (PC7)
- net PWM3: now also U1.CN10_2 (PC8)
- net PWM4: now also U1.CN10_1 (PC9)
- net PWM5: now also U1.CN7_28 (PA0)
- net PWM6: now also U1.CN7_30 (PA1)
- no-connect marks 71 -> 40
Other:
- note removed: "未使用"

Commit message: F446RE基板　シリアルサーボ用端子を4ピンに変更，GNDベタにビアを追加，ver 0.3
Parts:
- removed J14: Conn_01x02_Pin, OU_connector:DF1E-2P-2.5DS, symbol Connector:Conn_01x02_Pin
- added J14: Conn_01x04_Pin, OU_connector:DF1E-4P-2.5DS, symbol Connector:Conn_01x04_Pin
Connections:
- net +3.3V: now also J14.3 (Pin_3)
- net GND: now also J14.1 (Pin_1)
- net PA9: now also J14.2 (Pin_2)
- net PA10: now reaches U1.CN10_33 (PA10)
- net PA10: now also J14.4 (Pin_4)
- no-connect marks 40 -> 39

Commit message: F446RE基板　シリアル通信端子の電源ピンを5Vに変更，ver 0.5
Connections:
- net +3.3V: no longer J14.3 (Pin_3)
- net +5V: now also J14.3 (Pin_3)
Changed lines of the file:
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@@
-	)
-	(symbol
-		(lib_id "power:+3.3V")
-		(at 157.48 195.58 180)
-		(unit 1)
-		(body_style 1)
-		(exclude_from_sim no)
-		(in_bom yes)
-		(on_board yes)
-		(in_pos_files yes)
-		(dnp no)
-		(fields_autoplaced yes)
-		(property "Reference" "#PWR052"
-			(at 157.48 191.77 0)
-			(hide yes)
-			(show_name no)
-			(do_not_autoplace no)
-			(effects
-				(font
-					(size 1.27 1.27)
-				)
-			)
-		)
-		(property "Value" "+3.3V"
-			(at 157.48 200.66 0)
-			(show_name no)
-			(do_not_autoplace no)
-			(effects
-				(font
-					(size 1.27 1.27)
-				)
-			)
-		)
-		(property "Footprint" ""
-			(at 157.48 195.58 0)
-			(hide yes)
-			(show_name no)
-			(do_not_autoplace no)
-			(effects
-				(font
-					(size 1.27 1.27)
-				)
-			)
-		)
-		(property "Datasheet" ""
-			(at 157.48 195.58 0)
-			(hide yes)
-			(show_name no)
-			(do_not_autoplace no)
-			(effects
-				(font
-					(size 1.27 1.27)
-				)
-			)
-		)
-		(property "Description" "Power symbol creates a global label with name \"+3.3V\""
-			(at 157.48 195.58 0)
-			(hide yes)
-			(show_name no)
-			(do_not_autoplace no)
-			(effects
-				(font
-					(size 1.27 1.27)
-				)
-			)
-		)
-		(pin "1"
-		)
-		(instances
-			(project "Nucleo-F446RE_control_board"
-				(path "/831eb46c-8063-48af-b9d8-2e725b4cd87f"
-					(reference "#PWR052")
-					(unit 1)
-				)
-			)
-		)
 	)
 	(symbol
@@
 					(unit 1)
 				)
+			)
+		)
+	)
+	(symbol
+		(lib_id "power:+5V")
+		(at 157.48 195.58 180)
+		(unit 1)
+		(body_style 1)
+		(exclude_from_sim no)
+		(in_bom yes)
+		(on_board yes)
+		(in_pos_files yes)
+		(dnp no)
+		(fields_autoplaced yes)
+		(property "Reference" "#PWR047"
+			(at 157.48 191.77 0)
+			(hide yes)
+			(show_name no)
+			(do_not_autoplace no)
+			(effects
+				(font
+					(size 1.27 1.27)
+				)
+			)
+		)
+		(property "Value" "+5V"
+			(at 157.48 200.66 0)
+			(show_name no)
+			(do_not_autoplace no)
+			(effects
+				(font
+					(size 1.27 1.27)
+				)
+			)
+		)
+		(property "Footprint" ""
+			(at 157.48 195.58 0)
+			(hide yes)
+			(show_name no)
+			(do_not_autoplace no)
+			(effects
+				(font
+					(size 1.27 1.27)
+				)
+			)
+		)
+		(property "Datasheet" ""
+			(at 157.48 195.58 0)
+			(hide yes)
+			(show_name no)
+			(do_not_autoplace no)
+			(effects
+				(font
+					(size 1.27 1.27)
+				)
+			)
+		)
+		(property "Description" "Power symbol creates a global label with name \"+5V\""
+			(at 157.48 195.58 0)
+			(hide yes)
+			(show_name no)
+			(do_not_autoplace no)
+			(effects
+				(font
+					(size 1.27 1.27)
+				)
+			)
+		)
+		(pin "1"
+		)
+		(instances
+			(project "Nucleo-F446RE_control_board"
+				(path "/831eb46c-8063-48af-b9d8-2e725b4cd87f"
+					(reference "#PWR047")
+					(unit 1)
+				)
