File: micon_power_board/micon_power_board.kicad_pcb (KiCad board)
At the start: 2 copper layers, 55 x 45 mm, 27 parts, among them J1 Conn_01x02_Pin, J2 Conn_01x02_Pin, J3 Conn_01x02_Pin, J4 Conn_01x02_Pin, J5 Conn_01x02_Pin, J6 Conn_01x02_Pin, J7 Conn_01x02_Socket, U1 M78AR05-1

Commit message: マイコン電源基板　0.1uFのコンデンサの耐圧を他と揃えるため，変更，ver 0.7
Parts:
- C3: footprint Capacitor_THT:C_Disc_D4.7mm_W2.5mm_P5.00mm -> Capacitor_THT:C_Disc_D5.0mm_W2.5mm_P2.50mm
- moved C3 3.01 mm to (53.0, 26.4), turned to 180 degrees
Connections:
- C3 pad 1: Net-(D1-K) -> GND
- C3 pad 2: GND -> Net-(D1-K)
Routing:
- net Net-(D1-K): track 38.8 -> 39.3 mm
Other:
- board text added: "ver 0.7"
- board text removed: "ver 0.5"
Changed lines of the file:
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@@
 		(embedded_fonts no)
 	)
-	(footprint "Capacitor_THT:C_Disc_D4.7mm_W2.5mm_P5.00mm"
-		(layer "F.Cu")
-		(at 50.038 26.432)
-		(descr "C, Disc series, Radial, pin pitch=5.00mm, diameter*width=4.7*2.5mm^2, Capacitor, http://www.vishay.com/docs/45233/krseries.pdf")
-		(tags "C Disc series Radial pin pitch 5.00mm diameter 4.7mm width 2.5mm Capacitor")
-		(property "Reference" "C3"
-			(at -2.032 2.016 0)
-			(layer "F.SilkS")
-			(effects
-				(font
-					(size 1 1)
-					(thickness 0.15)
-				)
-			)
-		)
-		(property "Value" "0.1u"
-			(at 2.5 2.5 0)
-			(layer "F.Fab")
-			(effects
-				(font
-					(size 1 1)
-					(thickness 0.15)
-				)
-			)
-		)
-		(property "Datasheet" ""
-			(at 0 0 0)
-			(layer "F.Fab")
-			(hide yes)
-			(effects
-				(font
-					(size 1.27 1.27)
-				)
-			)
-		)
-		(property "Description" "0.1μF100V X7R"
-			(at 0 0 0)
-			(layer "F.Fab")
-			(hide yes)
-			(effects
-				(font
-					(size 1.27 1.27)
-				)
-			)
-		)
-		(property "KiLib_Generator" "capacitor/THT/other"
-			(at 0 0 0)
-			(layer "F.SilkS")
-			(hide yes)
-			(effects
-				(font
-					(size 1 1)
-					(thickness 0.15)
-				)
-			)
-		)
-		(property "Buy_URL" "https://akizukidenshi.com/catalog/g/g115927/"
-			(at 0 0 0)
-			(unlocked yes)
-			(layer "F.Fab")
-			(hide yes)
-			(effects
-				(font
-					(size 1 1)
-					(thickness 0.15)
-				)
-			)
-		)
-		(property ki_fp_filters "C_*")
-		(sheetname "/")
-		(sheetfile "micon_power_board.kicad_sch")
-		(units
-			(unit
-				(name "A")
-				(pins "1" "2")
-			)
-		)
-		(attr through_hole)
-		(duplicate_pad_numbers_are_jumpers no)
-		(fp_line
-			(start 0.03 -1.37)
-			(end 4.97 -1.37)
-			(stroke
-				(width 0.12)
-				(type solid)
-			)
-			(layer "F.SilkS")
-		)
-		(fp_line
-			(start 0.03 -1.04)
-			(end 0.03 -1.37)
-			(stroke
-				(width 0.12)
-				(type solid)
-			)
-			(layer "F.SilkS")
-		)
-		(fp_line
-			(start 0.03 1.37)
-			(end 0.03 1.04)
-			(stroke
-				(width 0.12)
-				(type solid)
-			)
-			(layer "F.SilkS")
-		)
-		(fp_line
-			(start 4.97 -1.37)
-			(end 4.97 -1.04)
-			(stroke
-				(width 0.12)
-				(type solid)
-			)
-			(layer "F.SilkS")
-		)
-		(fp_line
-			(start 4.97 1.04)
-			(end 4.97 1.37)
-			(stroke
-				(width 0.12)
-				(type solid)
-			)
-			(layer "F.SilkS")
-		)
-		(fp_line
-			(start 4.97 1.37)
-			(end 0.03 1.37)
-			(stroke
-				(width 0.12)
-				(type solid)
-			)
-			(layer "F.SilkS")
-		)
-		(fp_rect
-			(start -1.05 -1.5)
-			(end 6.05 1.5)
-			(stroke
-				(width 0.05)
-				(type solid)
-			)
-			(fill no)
-			(layer "F.CrtYd")
-		)
-		(fp_rect
-			(start 0.15 -1.25)
-			(end 4.85 1.25)
-			(stroke
-				(width 0.1)
-				(type solid)
-			)
-			(fill no)
-			(layer "F.Fab")
-		)
-		(fp_text user "${REFERENCE}"
-			(at 2.5 0 0)
-			(layer "F.Fab")
-			(effects
-				(font
-					(size 0.94 0.94)
-					(thickness 0.141)
-				)
-			)
-		)
-		(pad "1" thru_hole circle
-			(at 0 0)
-			(size 1.6 1.6)
-			(drill 0.8)
-			(layers "*.Cu" "*.Mask")
-			(remove_unused_layers no)
-			(net "Net-(D1-K)")
-			(pintype "passive")
-		)
-		(pad "2" thru_hole circle
-			(at 5 0)
-			(size 1.6 1.6)
-			(drill 0.8)
-			(layers "*.Cu" "*.Mask")
-			(remove_unused_layers no)
-			(net "GND")
-			(pintype "passive")
-		)
-		(embedded_fonts no)
-		(model "${KICAD10_3DMODEL_DIR}/Capacitor_THT.3dshapes/C_Disc_D4.7mm_W2.5mm_P5.00mm.step"
-			(offset
-				(xyz 0 0 0)
-			)
-			(scale
-				(xyz 1 1 1)
-			)
-			(rotate
-				(xyz 0 0 0)
-			)
-		)
-	)
 	(footprint "OU_connector:DF1E-2P-2.5DS"
 		(layer "F.Cu")
@@
 		)
 	)
+	(footprint "Capacitor_THT:C_Disc_D5.0mm_W2.5mm_P2.50mm"
+		(layer "F.Cu")
+		(at 53.046 26.416 180)
+		(descr "C, Disc series, Radial, pin pitch=2.50mm, diameter*width=5*2.5mm^2, Capacitor, http://cdn-reichelt.de/documents/datenblatt/B300/DS_KERKO_TC.pdf")
+		(tags "C Disc series Radial pin pitch 2.50mm diameter 5mm width 2.5mm Capacitor")
+		(property "Reference" "C3"
+			(at -2.58 0 0)
+			(layer "F.SilkS")
+			(effects
+				(font
+					(size 1 1)
+					(thickness 0.15)
+				)
+			)
+		)
+		(property "Value" "0.1u"
+			(at 1.25 2.5 0)
+			(layer "F.Fab")
+			(effects
+				(font
+					(size 1 1)
+					(thickness 0.15)
+				)
+			)
+		)
+		(property "Datasheet" ""
+			(at 0 0 0)
+			(layer "F.Fab")
+			(hide yes)
+			(effects
+				(font
+					(size 1.27 1.27)
+				)
+			)
+		)
+		(property "Description" "0.1μF50V X7R"
+			(at 0 0 0)
+			(layer "F.Fab")
+			(hide yes)
+			(effects
+				(font
+					(size 1.27 1.27)
+				)
+			)
+		)
+		(property "KiLib_Generator" "capacitor/THT/other"
+			(at 0 0 0)
+			(layer "F.SilkS")
+			(hide yes)
+			(effects
+				(font
+					(size 1 1)
+					(thickness 0.15)
+				)
+			)
+		)
+		(property "Buy_URL" "https://akizukidenshi.com/catalog/g/g113582/"
+			(at 0 0 180)
+			(unlocked yes)
+			(layer "F.Fab")
+			(hide yes)
+			(effects
+				(font
+					(size 1 1)
+					(thickness 0.15)
+				)
+			)
+		)
+		(property ki_fp_filters "C_*")
+		(sheetname "/")
+		(sheetfile "micon_power_board.kicad_sch")
+		(units
+			(unit
+				(name "A")
+				(pins "1" "2")
+			)
+		)
+		(attr through_hole)
+		(duplicate_pad_numbers_are_jumpers no)
+		(fp_line
+			(start 3.87 1.37)
+			(end -1.37 1.37)
+			(stroke
+				(width 0.12)
+				(type solid)
+			)
+			(layer "F.SilkS")
+		)
+		(fp_line
+			(start 3.87 -1.37)
+			(end 3.87 1.37)
+			(stroke
+				(width 0.12)
+				(type solid)
+			)
+			(layer "F.SilkS")
+		)
+		(fp_line
+			(start -1.37 1.37)
+			(end -1.37 -1.37)
+			(stroke
+				(width 0.12)
+				(type solid)
+			)
+			(layer "F.SilkS")
+		)
+		(fp_line
+			(start -1.37 -1.37)
+			(end 3.87 -1.37)
+			(stroke
+				(width 0.12)
+				(type solid)
+			)
+			(layer "F.SilkS")
+		)
+		(fp_rect
+			(start -1.5 -1.5)
+			(end 4 1.5)
+			(stroke
+				(width 0.05)
+				(type solid)
+			)
+			(fill no)
+			(layer "F.CrtYd")
+		)
+		(fp_rect
+			(start -1.25 -1.25)
+			(end 3.75 1.25)
+			(stroke
+				(width 0.1)
+				(type solid)
+			)
+			(fill no)
+			(layer "F.Fab")
+		)
+		(fp_text user "${REFERENCE}"
+			(at 1.25 0 0)
+			(layer "F.Fab")
+			(effects
+				(font
+					(size 1 1)
+					(thickness 0.15)
+				)
+			)
+		)
+		(pad "1" thru_hole circle
+			(at 0 0 180)
+			(size 1.6 1.6)
+			(drill 0.8)
+			(layers "*.Cu" "*.Mask")
+			(remove_unused_layers no)
+			(net "GND")
+			(pintype "passive")
+		)
+		(pad "2" thru_hole circle
+			(at 2.5 0 180)
+			(size 1.6 1.6)
+			(drill 0.8)
+			(layers "*.Cu" "*.Mask")
+			(remove_unused_layers no)
+			(net "Net-(D1-K)")
+			(pintype "passive")
+		)
+		(embedded_fonts no)
+		(model "${KICAD10_3DMODEL_DIR}/Capacitor_THT.3dshapes/C_Disc_D5.0mm_W2.5mm_P2.50mm.step"
+			(offset
+				(xyz 0 0 0)
+			)
+			(scale
+				(xyz 1 1 1)
+			)
+			(rotate
+				(xyz 0 0 0)
+			)
+		)
+	)
 	(footprint "LED_THT:LED_D5.0mm"
 		(layer "F.Cu")
@@
 		)
 	)
-	(gr_text "ver 0.5"
+	(gr_text "ver 0.7"
 		(at 68.8 55.8 0)
 		(layer "F.SilkS")
@@
 	)
 	(segment
-		(start 39.116 26.686)
-		(end 36.576 24.146)
+		(start 50.837999 22.389999)
+		(end 50.837999 26.124001)
 		(width 0.25)
 		(layer "B.Cu")
@@
 	)
 	(segment
-		(start 50.038 26.432)
-		(end 50.038 31.004)
+		(start 39.116 26.686)
+		(end 36.576 24.146)
 		(width 0.25)
 		(layer "B.Cu")
@@
 	)
 	(segment
+		(start 50.53 26.432)
+		(end 50.546 26.416)
+		(width 0.25)
+		(layer "B.Cu")
+		(net "Net-(D1-K)")
+	)
+	(segment
+		(start 50.292 21.844)
+		(end 50.837999 22.389999)
+		(width 0.25)
+		(layer "B.Cu")
+		(net "Net-(D1-K)")
+	)
+	(segment
 		(start 39.116 33.02)
 		(end 39.878 33.782)
@@
 	)
 	(segment
-		(start 50.837999 22.389999)
-		(end 50.292 21.844)
+		(start 44.45 26.432)
+		(end 50.53 26.432)
 		(width 0.25)
 		(layer "B.Cu")
@@
 	)
 	(segment
-		(start 50.038 26.432)
-		(end 50.837999 25.632001)
+		(start 50.837999 26.124001)
+		(end 50.546 26.416)
 		(width 0.25)
 		(layer "B.Cu")
@@
 	)
 	(segment
-		(start 44.45 26.432)
-		(end 50.038 26.432)
+		(start 50.546 26.416)
+		(end 50.546 30.496)
 		(width 0.25)
 		(layer "B.Cu")
@@
 	)
 	(segment
-		(start 50.837999 25.632001)
-		(end 50.837999 22.389999)
+		(start 50.546 30.496)
+		(end 50.038 31.004)
 		(width 0.25)
 		(layer "B.Cu")

Commit message: マイコン電源基板　シルクを一部修正，ver 1.0
Parts:
- renumbered TP3 to TP1, TP1 to TP2, TP2 to TP3
Other:
- board text added: "2026/10/10 Designed by E.Yoshioka"
- board text added: "ver 1.0"
- board text removed: "2026/09/24 Designed by E.Yoshioka"
- board text removed: "ver 0.7"
Changed lines of the file:
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@@
 		(descr "THT pad as test Point, diameter 2.0mm, hole diameter 1.0mm")
 		(tags "test point THT pad")
-		(property "Reference" "TP3"
+		(property "Reference" "TP1"
 			(at 3.048 -0.254 0)
 			(layer "F.SilkS")
@@
 		(descr "THT pad as test Point, diameter 2.0mm, hole diameter 1.0mm")
 		(tags "test point THT pad")
-		(property "Reference" "TP2"
+		(property "Reference" "TP3"
 			(at 1.016 -2.794 90)
 			(layer "F.SilkS")
@@
 		(descr "THT pad as test Point, diameter 2.0mm, hole diameter 1.0mm")
 		(tags "test point THT pad")
-		(property "Reference" "TP1"
+		(property "Reference" "TP2"
 			(at -3.048 0.508 0)
 			(layer "F.SilkS")
@@
 	)
 	(gr_rect
+		(start 42.204 57.698)
+		(end 47.204 62.698)
+		(stroke
+			(width 0)
+			(type solid)
+		)
+		(fill yes)
+		(layer "B.SilkS")
+	)
+	(gr_rect
 		(start 66.55 34.1)
 		(end 73.45 46.6)
@@
 		)
 	)
-	(gr_text "ver 0.7"
+	(gr_text "ver 1.0"
 		(at 68.8 55.8 0)
 		(layer "F.SilkS")
@@
 		)
 	)
-	(gr_text "2026/09/24\nDesigned by E.Yoshioka"
-		(at 49.784 60 0)
+	(gr_text "2026/10/10\nDesigned by E.Yoshioka"
+		(at 43.942 40.386 0)
 		(layer "B.SilkS")
 		(effects
