File: serial_servo_control_board/serial_servo_control_board.kicad_pcb (KiCad board)
At the start: 2 copper layers, 35 x 50 mm, 28 parts, among them J1 Conn_01x04_Pin, J2 Conn_01x02_Pin, J3 Conn_01x03_Pin, Q1 BSS138, Q2 BSS138, U1 NJM2884U2-05, U2 TLP2745, U3 TLP2745

Commit message: シリアルモータ制御基板　シルクを一部修正，ver 1.0
Parts:
- renumbered C5 to C2, C7 to C4, C6 to C5, D4 to D1, D5 to D2, R5 to R2, R4 to R3, R2 to R4, TP3 to TP1, TP4 to TP2, TP2 to TP3, TP1 to TP4
Routing:
- net GNDPWR: vias 45 -> 44
Other:
- board text added: "2026/10/10 Designed by E.Yoshioka"
- board text added: "ver 1.0"
- board text removed: "2026/10/09 Designed by E.Yoshioka"
- board text removed: "ver 0.1"
Changed lines of the file:
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@@
 		(descr "Diode, DO-34_SOD68 series, Axial, Vertical, pin pitch=2.54mm, length*diameter=3.04*1.6mm^2, https://www.nxp.com/docs/en/data-sheet/KTY83_SER.pdf")
 		(tags "Diode DO-34_SOD68 series Axial Vertical pin pitch 2.54mm  length 3.04mm diameter 1.6mm")
-		(property "Reference" "D5"
+		(property "Reference" "D2"
 			(at 5.08 0 0)
 			(layer "F.SilkS")
@@
 			(remove_unused_layers no)
 			(roundrect_rratio 0.166667)
-			(net "Net-(D5-K)")
+			(net "Net-(D2-K)")
 			(pinfunction "K_1")
 			(pintype "passive")
@@
 			(layers "*.Cu" "*.Mask")
 			(remove_unused_layers no)
-			(net "Net-(D4-K)")
+			(net "Net-(D1-K)")
 			(pinfunction "A_2")
 			(pintype "passive")
@@
 		(descr "THT pad as test Point, diameter 2.0mm, hole diameter 1.0mm")
 		(tags "test point THT pad")
-		(property "Reference" "TP3"
+		(property "Reference" "TP1"
 			(at 0 -1.998 0)
 			(layer "F.SilkS")
@@
 			)
 		)
+		(property "Buy_URL" "https://akizukidenshi.com/catalog/g/g104232/"
+			(at 0 0 180)
+			(unlocked yes)
+			(layer "F.Fab")
+			(hide yes)
+			(effects
+				(font
+					(size 1 1)
+					(thickness 0.15)
+				)
+			)
+		)
 		(property ki_fp_filters "SOT?23*")
 		(sheetname "/")
@@
 		(descr "Resistor, Axial_DIN0207 series, Axial, Vertical, pin pitch=2.54mm, 0.25W = 1/4W, length*diameter=6.3*2.5mm^2, http://cdn-reichelt.de/documents/datenblatt/B400/1_4W%23YAG.pdf")
 		(tags "Resistor Axial_DIN0207 series Axial Vertical pin pitch 2.54mm 0.25W = 1/4W length 6.3mm diameter 2.5mm")
-		(property "Reference" "R2"
+		(property "Reference" "R4"
 			(at 4.826 -1.27 90)
 			(layer "F.SilkS")
@@
 		(descr "Diode, DO-34_SOD68 series, Axial, Vertical, pin pitch=2.54mm, length*diameter=3.04*1.6mm^2, https://www.nxp.com/docs/en/data-sheet/KTY83_SER.pdf")
 		(tags "Diode DO-34_SOD68 series Axial Vertical pin pitch 2.54mm  length 3.04mm diameter 1.6mm")
-		(property "Reference" "D4"
+		(property "Reference" "D1"
 			(at 5.08 0 0)
 			(layer "F.SilkS")
@@
 			(remove_unused_layers no)
 			(roundrect_rratio 0.166667)
-			(net "Net-(D4-K)")
+			(net "Net-(D1-K)")
 			(pinfunction "K_1")
 			(pintype "passive")
@@
 			(layers "*.Cu" "*.Mask")
 			(remove_unused_layers no)
-			(net "Net-(D4-A)")
+			(net "Net-(D1-A)")
 			(pinfunction "A_2")
 			(pintype "passive")
@@
 		(descr "C, Disc series, Radial, pin pitch=2.50mm, diameter*width=5*2.5mm^2, Capacitor, http://cdn-reichelt.de/documents/datenblatt/B300/DS_KERKO_TC.pdf")
 		(tags "C Disc series Radial pin pitch 2.50mm diameter 5mm width 2.5mm Capacitor")
-		(property "Reference" "C7"
+		(property "Reference" "C4"
 			(at 3.262 2.286 90)
 			(layer "F.SilkS")
@@
 		(descr "C, Disc series, Radial, pin pitch=2.50mm, diameter*width=5*2.5mm^2, Capacitor, http://cdn-reichelt.de/documents/datenblatt/B300/DS_KERKO_TC.pdf")
 		(tags "C Disc series Radial pin pitch 2.50mm diameter 5mm width 2.5mm Capacitor")
-		(property "Reference" "C6"
+		(property "Reference" "C5"
 			(at -2.794 -1.524 0)
 			(layer "F.SilkS")
@@
 		(descr "THT pad as test Point, diameter 2.0mm, hole diameter 1.0mm")
 		(tags "test point THT pad")
-		(property "Reference" "TP1"
+		(property "Reference" "TP4"
 			(at 2.794 -1.016 0)
 			(layer "F.SilkS")
@@
 		(descr "THT pad as test Point, diameter 2.0mm, hole diameter 1.0mm")
 		(tags "test point THT pad")
-		(property "Reference" "TP2"
+		(property "Reference" "TP3"
 			(at 0 -1.998 0)
 			(layer "F.SilkS")
@@
 		(descr "THT pad as test Point, diameter 2.0mm, hole diameter 1.0mm")
 		(tags "test point THT pad")
-		(property "Reference" "TP4"
+		(property "Reference" "TP2"
 			(at 0 -1.998 0)
 			(layer "F.SilkS")
@@
 		(descr "CP, Radial series, Radial, pin pitch=5.00mm, diameter=10mm, height=16mm, Electrolytic Capacitor")
 		(tags "CP Radial series Radial pin pitch 5.00mm diameter 10mm height 16mm Electrolytic Capacitor")
-		(property "Reference" "C5"
+		(property "Reference" "C2"
 			(at 2.54 -6.096 0)
 			(layer "F.SilkS")
@@
 			(size 0.8 1.3)
 			(layers "F.Cu" "F.Mask" "F.Paste")
-			(net "Net-(D5-K)")
+			(net "Net-(D2-K)")
 			(pinfunction "A_1")
 			(pintype "passive")
@@
 		(descr "Resistor, Axial_DIN0207 series, Axial, Vertical, pin pitch=2.54mm, 0.25W = 1/4W, length*diameter=6.3*2.5mm^2, http://cdn-reichelt.de/documents/datenblatt/B400/1_4W%23YAG.pdf")
 		(tags "Resistor Axial_DIN0207 series Axial Vertical pin pitch 2.54mm 0.25W = 1/4W length 6.3mm diameter 2.5mm")
-		(property "Reference" "R5"
+		(property "Reference" "R2"
 			(at 4.826 0 0)
 			(layer "F.SilkS")
@@
 			(layers "*.Cu" "*.Mask")
 			(remove_unused_layers no)
-			(net "Net-(D4-A)")
+			(net "Net-(D1-A)")
 			(pintype "passive")
 		)
@@
 			)
 		)
+		(property "Buy_URL" "https://akizukidenshi.com/catalog/g/g104232/"
+			(at 0 0 0)
+			(unlocked yes)
+			(layer "F.Fab")
+			(hide yes)
+			(effects
+				(font
+					(size 1 1)
+					(thickness 0.15)
+				)
+			)
+		)
 		(property ki_fp_filters "SOT?23*")
 		(sheetname "/")
@@
 		(descr "Resistor, Axial_DIN0207 series, Axial, Vertical, pin pitch=2.54mm, 0.25W = 1/4W, length*diameter=6.3*2.5mm^2, http://cdn-reichelt.de/documents/datenblatt/B400/1_4W%23YAG.pdf")
 		(tags "Resistor Axial_DIN0207 series Axial Vertical pin pitch 2.54mm 0.25W = 1/4W length 6.3mm diameter 2.5mm")
-		(property "Reference" "R4"
+		(property "Reference" "R3"
 			(at 4.572 1.016 0)
 			(layer "F.SilkS")
@@
 	)
 	(gr_rect
+		(start 72.938 87.924)
+		(end 77.938 92.924)
+		(stroke
+			(width 0)
+			(type solid)
+		)
+		(fill yes)
+		(layer "B.SilkS")
+	)
+	(gr_rect
 		(start 55 50)
 		(end 90 100)
@@
 		)
 	)
-	(gr_text "ver 0.1"
+	(gr_text "ver 1.0"
 		(at 83.312 59.182 0)
 		(layer "F.SilkS")
@@
 		)
 	)
-	(gr_text "2026/10/09\nDesigned by E.Yoshioka"
+	(gr_text "2026/10/10\nDesigned by E.Yoshioka"
 		(at 81.28 61.214 90)
 		(layer "B.SilkS")
@@
 	)
 	(via
-		(at 75 92)
-		(size 0.8)
-		(drill 0.4)
-		(layers "F.Cu" "B.Cu")
-		(free yes)
-		(net "GNDPWR")
-	)
-	(via
 		(at 80 61)
 		(size 0.8)
@@
 	)
 	(segment
-		(start 78.486 93.116)
-		(end 78.334 92.964)
-		(width 0.25)
-		(layer "F.Cu")
-		(net "Net-(D5-K)")
-	)
-	(segment
-		(start 78.486 95.25)
-		(end 78.486 93.116)
-		(width 0.25)
-		(layer "F.Cu")
-		(net "Net-(D5-K)")
-	)
-	(segment
-		(start 75.946 97.79)
-		(end 75.946 95.25)
-		(width 0.25)
-		(layer "F.Cu")
-		(net "Net-(D4-K)")
-	)
-	(segment
 		(start 67.56 67.564)
 		(end 70.104 70.108)
@@
 		(width 0.25)
 		(layer "F.Cu")
-		(net "Net-(D4-A)")
+		(net "Net-(D1-A)")
 	)
 	(segment
@@
 		(width 0.25)
 		(layer "F.Cu")
-		(net "Net-(D4-A)")
+		(net "Net-(D1-A)")
+	)
+	(segment
+		(start 75.946 97.79)
+		(end 75.946 95.25)
+		(width 0.25)
+		(layer "F.Cu")
+		(net "Net-(D1-K)")
+	)
+	(segment
+		(start 78.486 93.116)
+		(end 78.334 92.964)
+		(width 0.25)
+		(layer "F.Cu")
+		(net "Net-(D2-K)")
+	)
+	(segment
+		(start 78.486 95.25)
+		(end 78.486 93.116)
+		(width 0.25)
+		(layer "F.Cu")
+		(net "Net-(D2-K)")
 	)
 	(zone
