File: serial_servo_control_board/serial_servo_control_board.kicad_sch (KiCad schematic)
At the start: 18 parts, among them J1 Conn_01x04_Pin, J2 Conn_01x02_Pin, J3 Conn_01x03_Pin, Q1 BSS138, Q2 BSS138, U1 NJM2884U2-05, U2 TLP2745, U3 TLP2745

Commit message: シリアルモータ制御基板　基板完成，ver 0.1
Parts:
- added R5: 47k, Resistor_THT:R_Axial_DIN0207_L6.3mm_D2.5mm_P2.54mm_Vertical, symbol Device:R
- added TP1, TP2: TestPoint_Probe, TestPoint:TestPoint_THTPad_D2.0mm_Drill1.0mm, symbol Connector:TestPoint_Probe
- added TP3, TP4: TestPoint, TestPoint:TestPoint_THTPad_D2.0mm_Drill1.0mm, symbol Connector:TestPoint
Connections:
- net GND: now also TP3.1
- net GNDPWR: now also R5.1, TP4.1
- net RX: now also TP2.1
- net signal: now also TP1.1
- net at Q2.1 (G), U2.5 (VO): now also R5.2
Other:
- note added: "6.0V"
- note removed: "5.0~7.4V"

Commit message: シリアルモータ制御基板　不足していた部品URLを追加
Parts:
- Q1, Q2: Buy_URL (none) -> https://akizukidenshi.com/catalog/g/g104232/
Changed lines of the file:
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@@
+			)
+		)
+		(property "Buy_URL" "https://akizukidenshi.com/catalog/g/g104232/"
+			(at 119.38 92.71 0)
+			(hide yes)
+			(show_name no)
+			(do_not_autoplace no)
+			(effects
+				(font
+					(size 1.27 1.27)
+				)
 			)
 		)
@@
 			(at 125.73 38.1 0)
 			(hide yes)
+			(show_name no)
+			(do_not_autoplace no)
+			(effects
+				(font
+					(size 1.27 1.27)
+				)
+			)
+		)
+		(property "Buy_URL" "https://akizukidenshi.com/catalog/g/g104232/"
+			(at 125.73 38.1 0)
+			(hide yes)

Commit message: シリアルモータ制御基板　シルクを一部修正，ver 1.0
Parts:
- renumbered C5 to C2, C7 to C4, C6 to C5, D4 to D1, D5 to D2, R5 to R2, R4 to R3, R2 to R4, TP3 to TP1, TP4 to TP2, TP2 to TP3, TP1 to TP4
